File: ESP32-S3-WROOM-1/ESP32-S3-WROOM-1.kicad_sch (KiCad schematic)
At the start: 23 parts, among them J1 ESP32-S3-DEVKITC-1-J1, J2 ESP32-S3-DEVKITC-1-J2, J3 UART, P1 USB2.0_C_12pin, SW1 SW_Push, SW2 SW_Push, U1 ESP32-S3-WROOM-1, U2 AMS1117-3.3

Commit message: 漏れ
Parts:
- removed C7: 100n, Capacitor_SMD:C_0805_2012Metric_Pad1.18x1.45mm_HandSolder, symbol Device:C
- added R4: 10k, Resistor_SMD:R_0805_2012Metric_Pad1.20x1.40mm_HandSolder, symbol Device:R
- D1: value LED -> 5V
- D2: value LED -> D-
- D3: value LED -> D+
- D5: value LED -> PWR
- SW1: value SW_Push -> BOOT
- SW2: value SW_Push -> RESET
Connections:
- net +3V3: now also R4.2
- net CHIP_PU: now also C2.1, R4.1
- net GPIO0: no longer C2.1

Commit message: 漏れ
Connections:
- net VBUS: no longer names the net of D1.2 (A), D4.2 (A), P1.11 (VBUS_B4/A9), P1.2 (VBUS_A4/B9)
Changed lines of the file:
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@@
   (junction (at 210.82 144.78) (diameter 0) (color 0 0 0 0)
-  )
-  (junction (at 93.98 45.72) (diameter 0) (color 0 0 0 0)
   )
   (junction (at 210.82 137.16) (diameter 0) (color 0 0 0 0)
@@
     (stroke (width 0) (type default) (color 0 0 0 0))
   )
-  (wire (pts (xy 93.98 45.72) (xy 104.14 45.72))
-    (stroke (width 0) (type default) (color 0 0 0 0))
-  )
   (wire (pts (xy 124.46 71.12) (xy 127 71.12))
     (stroke (width 0) (type default) (color 0 0 0 0))
@@
     (stroke (width 0) (type default) (color 0 0 0 0))
   )
-  (wire (pts (xy 93.98 38.1) (xy 93.98 45.72))
-    (stroke (width 0) (type default) (color 0 0 0 0))
-  )
   (wire (pts (xy 67.31 66.04) (xy 72.39 66.04))
     (stroke (width 0) (type default) (color 0 0 0 0))
@@
     (stroke (width 0) (type default) (color 0 0 0 0))
   )
-  (wire (pts (xy 72.39 45.72) (xy 93.98 45.72))
+  (wire (pts (xy 72.39 45.72) (xy 104.14 45.72))
     (stroke (width 0) (type default) (color 0 0 0 0))
   )
@@
     (pin "5")
     (pin "6")
-  )
-  (symbol (lib_id "power:VBUS") (at 93.98 38.1 0) (unit 1)
-    (in_bom yes) (on_board yes) (fields_autoplaced)
-    (property "Reference" "#PWR04" (id 0) (at 93.98 41.91 0)
-      (effects (font (size 1.27 1.27)) hide)
-    )
-    (property "Value" "VBUS" (id 1) (at 93.98 33.02 0))
-    (property "Footprint" "" (id 2) (at 93.98 38.1 0)
-      (effects (font (size 1.27 1.27)) hide)
-    )
-    (property "Datasheet" "" (id 3) (at 93.98 38.1 0)
-      (effects (font (size 1.27 1.27)) hide)
-    )
-    (pin "1")
   )
   (symbol (lib_id "power:GND") (at 96.52 81.28 0) (unit 1)
@@
       (reference "#PWR03") (unit 1) (value "GND") (footprint "")
     )
-    (path "/7fb86b8e-60bd-46f2-8f11-74cbd3a85915"
-      (reference "#PWR04") (unit 1) (value "VBUS") (footprint "")
-    )
     (path "/839ff533-2dd2-43cc-a86a-db4150544962"
