File: ESP32-S3-WROOM-1/ESP32-S3-WROOM-1.kicad_sch (KiCad schematic)
At the start: 23 parts, among them J1 ESP32-S3-DEVKITC-1-J1, J2 ESP32-S3-DEVKITC-1-J2, J3 UART, P1 USB2.0_C_12pin, SW1 BOOT, SW2 RESET, U1 ESP32-S3-WROOM-1, U2 AMS1117-3.3

Commit message: fix
Parts:
- removed P1: USB2.0_C_12pin, esp32-dev-boards:USB-C-12-Pin-MidMount, symbol $74th:USB2.0_C_12pin
- added J4: USB2.0_C_v3, $74th:USB-C-12-Pin-MidMount-ali-v4, symbol $74th:USB2.0_C_v3
Connections:
- net GND: now also J4.4 (GND)
- net GPIO19: now also D2.2 (A), J4.2 (D-); no longer D3.2 (A)
- net GPIO20: now also D3.2 (A), J4.3 (D+); no longer D2.2 (A)
- net at D1.2 (A), D4.2 (A): now also J4.1 (VBUS)
- net at R1.1: now also J4.6 (CC2)
- net at R2.1: now also J4.5 (CC1)
- no-connect marks 2 -> 0
Other:
- moved on the sheet: C1, D4

Commit message: up
Parts:
- removed J3: UART, esp32-dev-boards:UART, symbol esp32-dev-boards:UART
- added J3: ESP-Prog-ProgramCOM-RECV, $74th:BoxPinHeader_2x03_P1.27mm_Vertical, symbol $74th:ESP-Prog-ProgramCOM-RECV
- C1, C3, C4, C5, C6: footprint Capacitor_SMD:C_0805_2012Metric_Pad1.18x1.45mm_HandSolder -> esp32-dev-boards:Capacitor_0805_2012
- C2: value 100n -> 1u; footprint Capacitor_SMD:C_0805_2012Metric_Pad1.18x1.45mm_HandSolder -> esp32-dev-boards:Capacitor_0805_2012
- R1, R2, R4: footprint Resistor_SMD:R_0805_2012Metric_Pad1.20x1.40mm_HandSolder -> esp32-dev-boards:Register_0805_2012
- R3: value 5.1k -> 1k; footprint Resistor_SMD:R_0805_2012Metric_Pad1.20x1.40mm_HandSolder -> esp32-dev-boards:Register_0805_2012
Connections:
- net +5V: now also J3.2 (VCC)
- net CHIP_PU: now also J3.1 (EN)
- net GND: now also J3.4 (GND)
- net GPIO0: now also J3.6 (IO0)
- net U0RXD: now also J3.3 (RXD0)
- net U0TXD: now also J3.5 (TXD0)

Commit message: ESP32-C3-WROOM-02
Connections:
- net U0RXD: now also J3.5 (RXD0); no longer J3.3 (RXD0)
- net U0TXD: now also J3.3 (TXD0); no longer J3.5 (TXD0)
Changed lines of the file:
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@@
     )
   )
-  (global_label "U0TXD" (shape input) (at 246.38 62.23 0) (fields_autoplaced)
-    (effects (font (size 1.27 1.27)) (justify left))
-    (property "Intersheet References" "${INTERSHEET_REFS}" (id 0) (at 254.7802 62.1506 0)
+  (global_label "U0TXD" (shape input) (at 246.38 59.69 0) (fields_autoplaced)
+    (effects (font (size 1.27 1.27)) (justify left))
+    (property "Intersheet References" "${INTERSHEET_REFS}" (id 0) (at 254.7802 59.6106 0)
       (effects (font (size 1.27 1.27)) (justify left) hide)
     )
@@
     )
   )
-  (global_label "U0RXD" (shape input) (at 246.38 59.69 0) (fields_autoplaced)
-    (effects (font (size 1.27 1.27)) (justify left))
-    (property "Intersheet References" "${INTERSHEET_REFS}" (id 0) (at 255.0826 59.6106 0)
+  (global_label "U0RXD" (shape input) (at 246.38 62.23 0) (fields_autoplaced)
+    (effects (font (size 1.27 1.27)) (justify left))
+    (property "Intersheet References" "${INTERSHEET_REFS}" (id 0) (at 255.0826 62.1506 0)
       (effects (font (size 1.27 1.27)) (justify left) hide)
     )
@@
       (effects (font (size 1.27 1.27)) hide)
     )
-    (property "Datasheet" "" (id 3) (at 242.57 109.22 0)
+    (property "Datasheet" "~" (id 3) (at 242.57 109.22 0)
       (effects (font (size 1.27 1.27)) hide)
     )
@@
       (effects (font (size 1.27 1.27)) hide)
     )
-    (property "Datasheet" "" (id 3) (at 86.36 129.54 0)
-      (effects (font (size 1.27 1.27)) hide)
-    )
+    (property "Datasheet" "https://www.espressif.com/sites/default/files/documentation/esp32-s3-wroom-1_wroom-1u_datasheet_en.pdf" (id 3) (at 86.36 129.54 0)
+      (effects (font (size 1.27 1.27)) hide)
+    )

Commit message: fix D1, IO14
Parts:
- added R1: 1k, esp32-dev-boards:Register_0805_2012, symbol Device:R
- SW1: value BOOT -> BT
- SW2: value RESET -> RST
- renumbered C3 to C2, C4 to C3, C5 to C4, C6 to C5, C2 to C6, D4 to D1, D1 to D2, D2 to D3, D3 to D4, J4 to J3, J3 to J4, R1 to R2, R2 to R3, R3 to R4, R4 to R5, U2 to U1, U1 to U2
Connections:
- net +5V: now also R1.2
- net at D1.2 (A), J3.1 (VBUS): no longer D2.2 (A)
- new net: D2.2 (A), R1.1
Other:
- moved on the sheet: C1, D1, D2, D3, D4

Commit message: new ver
Parts:
- removed D2: 5V, LED_SMD:LED_0805_2012Metric_Pad1.15x1.40mm_HandSolder, symbol Device:LED
- removed D3: D-, LED_SMD:LED_0805_2012Metric_Pad1.15x1.40mm_HandSolder, symbol Device:LED
- removed D4: D+, LED_SMD:LED_0805_2012Metric_Pad1.15x1.40mm_HandSolder, symbol Device:LED
- removed R1: 1k, esp32-dev-boards:Register_0805_2012, symbol Device:R
- J1: footprint esp32-dev-boards:ESP32-S3-DEVKITC-J1 -> esp32-dev-boards:ESP32-S3-DEVKITC-J1-mini; symbol esp32-dev-boards:ESP32-S3-DEVKITC-1-J1 -> esp32-dev-boards:ESP32-S3-DEVKITC-1-J1-mini
- J2: footprint esp32-dev-boards:ESP32-S3-DEVKITC-J2 -> esp32-dev-boards:ESP32-S3-DEVKITC-J2-mini; symbol esp32-dev-boards:ESP32-S3-DEVKITC-1-J2 -> esp32-dev-boards:ESP32-S3-DEVKITC-1-J2-mini
- J4: renamed from J3; footprint $74th:USB-C-12-Pin-MidMount-ali-v4 -> $74th:USB-C-12-Pin-SMD
- SW1: renamed from SW2; value RST -> RS
- renumbered C6 to C1, C5 to C2, C4 to C3, C1 to C4, C2 to C5, C3 to C6, D5 to D1, D1 to D2, J4 to J3, R5 to R1, R4 to R2, R2 to R3, R3 to R4, SW1 to SW2, U2 to U1, U1 to U2
Connections:
- net +3V3: no longer J1.1 (ESP_3V3)
- net GND: no longer J1.22 (GND), J2.1 (GND), J2.22 (GND)
Other:
- moved on the sheet: C4, D2, SW1

Commit message: new ver
Parts:
- removed C4: 10u, esp32-dev-boards:Capacitor_0805_2012, symbol Device:C
- C1: value 1u -> 100n
Connections:
- net GND is gone; now on net +5V: C1.2, C2.2, C3.2, C5.2, C6.2, D1.1 (K), J2.21 (GND), J3.4 (GND), J4.4 (GND), R3.2, R4.2, SW1.1, SW2.1, U1.1 (GND), U1.40 (GND), U1.41 (GND), U2.1 (GND)
Changed lines of the file:
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@@
       (effects (font (size 1.27 1.27)) (justify left))
     )
-    (property "Value" "1u" (at 171.45 153.6699 0)
+    (property "Value" "100n" (at 171.45 153.6699 0)
       (effects (font (size 1.27 1.27)) (justify left))
     )
@@
     )
   )
-  (symbol (lib_id "power:GND") (at 96.52 50.8 0) (unit 1)
-    (in_bom yes) (on_board yes) (dnp no) (fields_autoplaced)
-    (property "Reference" "#PWR04" (at 96.52 57.15 0)
-      (effects (font (size 1.27 1.27)) hide)
-    )
-    (property "Value" "GND" (at 96.52 55.88 0)
-      (effects (font (size 1.27 1.27)))
-    )
-    (property "Footprint" "" (at 96.52 50.8 0)
-      (effects (font (size 1.27 1.27)) hide)
-    )
-    (property "Datasheet" "" (at 96.52 50.8 0)
+  (symbol (lib_id "power:GND") (at 96.52 43.18 0) (unit 1)
+    (in_bom yes) (on_board yes) (dnp no) (fields_autoplaced)
+    (property "Reference" "#PWR04" (at 96.52 49.53 0)
+      (effects (font (size 1.27 1.27)) hide)
+    )
+    (property "Value" "GND" (at 96.52 48.26 0)
+      (effects (font (size 1.27 1.27)))
+    )
+    (property "Footprint" "" (at 96.52 43.18 0)
+      (effects (font (size 1.27 1.27)) hide)
+    )
+    (property "Datasheet" "" (at 96.52 43.18 0)
       (effects (font (size 1.27 1.27)) hide)
     )
@@
         )
       )
-    )
-  )
-  (symbol (lib_id "Device:C") (at 96.52 46.99 0) (unit 1)
-    (in_bom yes) (on_board yes) (dnp no) (fields_autoplaced)
-    (property "Reference" "C4" (at 100.33 45.7199 0)
-      (effects (font (size 1.27 1.27)) (justify left))
-    )
-    (property "Value" "10u" (at 100.33 48.2599 0)
-      (effects (font (size 1.27 1.27)) (justify left))
-    )
-    (property "Footprint" "esp32-dev-boards:Capacitor_0805_2012" (at 97.4852 50.8 0)
-      (effects (font (size 1.27 1.27)) hide)
-    )
-    (property "Datasheet" "~" (at 96.52 46.99 0)
-      (effects (font (size 1.27 1.27)) hide)
-    )
-    (pin "1")
-    (pin "2")
-    (instances
-      (project "ESP32-S3-WROOM-1"
-        (path "/1f0126c3-e865-4b7c-bf68-4d53d0d38c5a"
-          (reference "C4") (unit 1)
-        )
-      )

Commit message: v1.2.0
Parts:
- C3: renamed from C1; value 100n -> 1u
- renumbered C3 to C1, C6 to C4, R4 to R3, R3 to R4
Changed lines of the file:
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@@
   (symbol (lib_id "Device:R") (at 67.31 71.12 0) (unit 1)
     (in_bom yes) (on_board yes) (dnp no) (fields_autoplaced)
-    (property "Reference" "R3" (at 69.85 69.8499 0)
+    (property "Reference" "R4" (at 69.85 69.8499 0)
       (effects (font (size 1.27 1.27)) (justify left))
     )
@@
       (project "ESP32-S3-WROOM-1"
         (path "/1f0126c3-e865-4b7c-bf68-4d53d0d38c5a"
-          (reference "R3") (unit 1)
+          (reference "R4") (unit 1)
         )
       )
@@
   (symbol (lib_id "Device:C") (at 167.64 152.4 0) (unit 1)
     (in_bom yes) (on_board yes) (dnp no) (fields_autoplaced)
-    (property "Reference" "C1" (at 171.45 151.1299 0)
-      (effects (font (size 1.27 1.27)) (justify left))
-    )
-    (property "Value" "100n" (at 171.45 153.6699 0)
+    (property "Reference" "C3" (at 171.45 151.1299 0)
+      (effects (font (size 1.27 1.27)) (justify left))
+    )
+    (property "Value" "1u" (at 171.45 153.6699 0)
       (effects (font (size 1.27 1.27)) (justify left))
     )
@@
       (project "ESP32-S3-WROOM-1"
         (path "/1f0126c3-e865-4b7c-bf68-4d53d0d38c5a"
-          (reference "C1") (unit 1)
+          (reference "C3") (unit 1)
         )
       )
@@
   (symbol (lib_id "Device:R") (at 77.47 71.12 0) (unit 1)
     (in_bom yes) (on_board yes) (dnp no) (fields_autoplaced)
-    (property "Reference" "R4" (at 80.01 69.8499 0)
+    (property "Reference" "R3" (at 80.01 69.8499 0)
       (effects (font (size 1.27 1.27)) (justify left))
     )
@@
       (project "ESP32-S3-WROOM-1"
         (path "/1f0126c3-e865-4b7c-bf68-4d53d0d38c5a"
-          (reference "R4") (unit 1)
+          (reference "R3") (unit 1)
         )
       )
@@
   (symbol (lib_id "Device:C") (at 218.44 109.22 0) (unit 1)
     (in_bom yes) (on_board yes) (dnp no) (fields_autoplaced)
-    (property "Reference" "C3" (at 222.25 107.9499 0)
+    (property "Reference" "C1" (at 222.25 107.9499 0)
       (effects (font (size 1.27 1.27)) (justify left))
     )
@@
       (project "ESP32-S3-WROOM-1"
         (path "/1f0126c3-e865-4b7c-bf68-4d53d0d38c5a"
-          (reference "C3") (unit 1)
+          (reference "C1") (unit 1)
         )
       )
@@
   (symbol (lib_id "Device:C") (at 189.23 109.22 0) (unit 1)
     (in_bom yes) (on_board yes) (dnp no) (fields_autoplaced)
-    (property "Reference" "C6" (at 193.04 107.9499 0)
+    (property "Reference" "C4" (at 193.04 107.9499 0)
       (effects (font (size 1.27 1.27)) (justify left))
     )
@@
       (project "ESP32-S3-WROOM-1"
         (path "/1f0126c3-e865-4b7c-bf68-4d53d0d38c5a"
-          (reference "C6") (unit 1)
-        )
-      )
+          (reference "C4") (unit 1)
+        )
+      )

Commit message: add title
Other:
- note added: "Button"
- note added: "ESP32-S3 Module"
- note added: "Pinout"
- note added: "Power"
- note added: "Program Port"
- note added: "USB"
- title: (none) -> ESP32-S3 Dev Board
- moved on the sheet: C1, C2, C3, C4, C5, D1, D2, J1, J2, J3, J4, R1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
