File: ESP32-C3-MINI-1/ESP32-C3-MINI-1.kicad_pcb (KiCad board)
At the start: 2 copper layers, 20.3 x 38.7 mm, 15 parts, among them J1 ESP32-C3-DEVKITM-1-J1, J2 ESP32-C3-DEVKITM-1-J2, J3 UART, SW1 BOOT, SW2 RESET, U1 ESP32-C3-MINI-1, U2 AMS1117-3.3

Commit message: order
Routing:
- net GPIO19: track 31.6 -> 30.5 mm
- net CHIP_PU: track 48.2 -> 47.5 mm
- net +3V3: track 55.8 -> 55.1 mm
