File: ESP32-C3-MINI-1/ESP32-C3-MINI-1.kicad_pcb (KiCad board)
At the start: 2 copper layers, 20.3 x 38.7 mm, 15 parts, among them J1 ESP32-C3-DEVKITM-1-J1, J2 ESP32-C3-DEVKITM-1-J2, J3 UART, SW1 BOOT, SW2 RESET, U1 ESP32-C3-MINI-1, U2 AMS1117-3.3

Commit message: fix
Other:
- board size 20.3 x 38.7 mm -> 20.3 x 44 mm

Commit message: up
Parts:
- added J4: USB2.0_C, esp32-dev-boards:USB-C-12-Pin-MidMount, F.Cu at (99.1, 116.0)
- added R2: 5.1k, Resistor_SMD:R_0805_2012Metric_Pad1.20x1.40mm_HandSolder, F.Cu at (131.3, 116.5)
- added R4: 5.1k, Resistor_SMD:R_0805_2012Metric_Pad1.20x1.40mm_HandSolder, F.Cu at (131.3, 119.5)
- added REF**: JLCJLCJLCJLC, $74th:JLCJLCJLCJLC, F.Cu at (97.9, 86.7)
- J3: value UART -> ESPProg-UART; footprint esp32-dev-boards:UART -> esp32-dev-boards:BoxPinHeader_2x03_P1.27mm_Vertical
- R3: value 5.1k -> 1k
- U1: footprint esp32-dev-boards:ESP32-C3-MINI-1 -> Espressif:ESP32-C3-MINI-1_Hand-Soldering
- moved C4 18.2 mm to (116.9, 104.8)
- moved C3 18.2 mm to (113.1, 104.9)
- moved C1 17.0 mm to (116.8, 109.9)
- moved R1 17.0 mm to (113.0, 109.9)
- moved C5 17.0 mm to (111.6, 96.6)
- moved C6 17.0 mm to (115.6, 96.6)
- moved R3 17.0 mm to (119.9, 99.4)
- moved SW2 15.5 mm to (95.7, 99.8)
- moved SW1 15.5 mm to (102.3, 99.8)
- moved J3 11.7 mm to (98.3, 111.2), turned to 90 degrees
- moved D5 1.64 mm to (104.9, 105.9)
- moved U2 1.43 mm to (99.0, 104.8)
Connections:
- J3 pad 1: U0TXD -> CHIP_PU
- J3 pad 2: U0RXD -> +5V
- J3 pad 3: +5V -> U0TXD
- J3 pad 5: CHIP_PU -> U0RXD
- R3 pad 2: +3V3 -> +5V
Routing:
- net +3V3: track 55.1 -> 0.00 mm
- net CHIP_PU: track 47.5 -> 0.00 mm, vias 1 -> 0
- net U0TXD: track 47.0 -> 0.00 mm
- net GPIO0: track 46.2 -> 0.00 mm, vias 1 -> 0
- net U0RXD: track 44.7 -> 0.00 mm
- net GPIO19: track 30.5 -> 0.00 mm, vias 1 -> 0
- net +5V: track 28.3 -> 0.00 mm
- net GPIO18: track 26.7 -> 0.00 mm, vias 1 -> 0
- net GPIO4: track 21.4 -> 0.00 mm
- net GPIO10: track 21.1 -> 0.00 mm
- net GPIO5: track 18.7 -> 0.00 mm
- net GPIO6: track 16.1 -> 0.00 mm
- net GPIO1: track 15.9 -> 0.00 mm
- net GPIO7: track 13.2 -> 0.00 mm
- net GPIO8: track 7.73 -> 0.00 mm
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Other:
- board text added: "ESP32C3 MINIDevBoard v1.1.0"
- board text removed: "GND"

Commit message: C3-MINI-1
Parts:
- added C2: 10u, Capacitor_SMD:C_0805_2012Metric_Pad1.18x1.45mm_HandSolder, B.Cu at (97.2, 86.9)
- C1, C3, C4, R1, R2, R3, R4: moved to B.Cu
- C5: value 10u -> 100n; moved to B.Cu
- C6: value 100n -> 10u; moved to B.Cu
- J4: footprint esp32-dev-boards:USB-C-12-Pin-MidMount -> esp32-dev-boards:USB-C-12-Pin-MidMount-ali-v4
- moved R4 36.4 mm to (95.3, 113.8)
- moved R2 28.2 mm to (103.2, 114.1), turned to 180 degrees
- moved C1 22.6 mm to (94.2, 109.7), turned to 180 degrees
- moved R1 18.9 mm to (94.2, 111.8)
- moved R3 17.7 mm to (102.9, 104.3), turned to -90 degrees
- moved C4 17.0 mm to (100.0, 106.7)
- moved C6 16.3 mm to (100.0, 101.3)
- moved C3 13.6 mm to (100.0, 108.8)
- moved C5 13.4 mm to (100.0, 103.4), turned to 0 degrees
- moved D5 1.42 mm to (104.6, 104.5)
Routing:
- net GPIO19: track 0.00 -> 47.0 mm, vias 0 -> 5
- net GPIO18: track 0.00 -> 46.8 mm, vias 0 -> 2
- net +3V3: track 0.00 -> 46.7 mm, vias 0 -> 3
- net U0TXD: track 0.00 -> 38.8 mm
- net GND: track 0.00 -> 38.4 mm, vias 0 -> 9
- net GPIO0: track 0.00 -> 38.2 mm, vias 0 -> 3
- net +5V: track 0.00 -> 37.9 mm, vias 0 -> 1
- net U0RXD: track 0.00 -> 36.0 mm, vias 0 -> 1
- net CHIP_PU: track 0.00 -> 33.8 mm, vias 0 -> 1
- net GPIO4: track 0.00 -> 26.3 mm, vias 0 -> 1
- net GPIO5: track 0.00 -> 22.9 mm, vias 0 -> 1
- net GPIO10: track 0.00 -> 19.0 mm, vias 0 -> 1
- net GPIO1: track 0.00 -> 15.7 mm, vias 0 -> 1
- net GPIO6: track 0.00 -> 15.5 mm
- net GPIO7: track 0.00 -> 13.0 mm
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Other:
- board size 20.3 x 44 mm -> 20.3 x 38.7 mm
- board text added: "ESP32C3 DevBoardM"
- board text added: "v1.1.0"
- board text removed: "ESP32C3 MINIDevBoard v1.1.0"
