File: ESP32-C3-MINI-1/ESP32-C3-MINI-1.kicad_sch (KiCad schematic)
At the start: 15 parts, among them J1 ESP32-C3-DEVKITM-1-J1, J2 ESP32-C3-DEVKITM-1-J2, J3 UART, SW1 BOOT, SW2 RESET, U1 ESP32-C3-MINI-1, U2 AMS1117-3.3

Commit message: up
Parts:
- removed J3: UART, esp32-dev-boards:UART, symbol esp32-dev-boards:UART
- added J3: ESPProg-UART, esp32-dev-boards:BoxPinHeader_2x03_P1.27mm_Vertical, symbol esp32-dev-boards:ESPProg-UART
- added J4: USB2.0_C, esp32-dev-boards:USB-C-12-Pin-MidMount, symbol esp32-dev-boards:USB2.0_C
- added R2, R4: 5.1k, Resistor_SMD:R_0805_2012Metric_Pad1.20x1.40mm_HandSolder, symbol Device:R
- R3: value 5.1k -> 1k
- U1: footprint esp32-dev-boards:ESP32-C3-MINI-1 -> Espressif:ESP32-C3-MINI-1_Hand-Soldering
Connections:
- net +3V3: no longer R3.2
- net +5V: now also R3.2, J3.2 (VCC), J4.1 (VBUS)
- net CHIP_PU: now also J3.1 (ESP_EN)
- net GND: now also J3.4 (GND), J4.4 (GND), R2.1, R4.1
- net GPIO0: now also J3.6 (ESP_BOOT)
- net GPIO18: now also J4.2 (D-)
- net GPIO19: now also J4.3 (D+)
- net U0RXD: now also J3.5 (ESP_RXD)
- net U0TXD: now also J3.3 (ESP_TXD)
- new net: J4.6 (CC2), R2.2
- new net: J4.5 (CC1), R4.2
Other:
- moved on the sheet: D5, R3

Commit message: C3-MINI-1
Parts:
- added C2: 10u, Capacitor_SMD:C_0805_2012Metric_Pad1.18x1.45mm_HandSolder, symbol Device:C
- C5: value 10u -> 100n
- C6: value 100n -> 10u
- J4: footprint esp32-dev-boards:USB-C-12-Pin-MidMount -> esp32-dev-boards:USB-C-12-Pin-MidMount-ali-v4
Connections:
- net +3V3: now also C2.1
- net GND: now also C2.2
Changed lines of the file:
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@@
 (kicad_sch (version 20211123) (generator eeschema)
   (paper "A4")
+  (junction (at 43.18 166.37) (diameter 0) (color 0 0 0 0)
+  )
   (junction (at 204.47 43.18) (diameter 0) (color 0 0 0 0)
   )
@@
     (stroke (width 0) (type default) (color 0 0 0 0))
   )
+  (wire (pts (xy 43.18 166.37) (xy 49.53 166.37))
+    (stroke (width 0) (type default) (color 0 0 0 0))
+  )
   (wire (pts (xy 67.31 73.66) (xy 67.31 71.12))
     (stroke (width 0) (type default) (color 0 0 0 0))
@@
     (stroke (width 0) (type default) (color 0 0 0 0))
   )
-  (wire (pts (xy 35.56 166.37) (xy 49.53 166.37))
+  (wire (pts (xy 35.56 166.37) (xy 43.18 166.37))
     (stroke (width 0) (type default) (color 0 0 0 0))
   )
@@
       (effects (font (size 1.27 1.27)) (justify left))
     )
-    (property "Value" "100n" (id 1) (at 247.65 48.2599 0)
+    (property "Value" "10u" (id 1) (at 247.65 48.2599 0)
       (effects (font (size 1.27 1.27)) (justify left))
     )
@@
       (effects (font (size 1.27 1.27)) (justify left))
     )
-    (property "Value" "10u" (id 1) (at 237.49 48.2599 0)
+    (property "Value" "100n" (id 1) (at 237.49 48.2599 0)
       (effects (font (size 1.27 1.27)) (justify left))
     )
@@
     (pin "1")
     (pin "2")
+  )
+  (symbol (lib_id "power:GND") (at 43.18 173.99 0) (unit 1)
+    (in_bom yes) (on_board yes) (fields_autoplaced)
+    (property "Reference" "#PWR08" (id 0) (at 43.18 180.34 0)
+      (effects (font (size 1.27 1.27)) hide)
+    )
+    (property "Value" "GND" (id 1) (at 43.18 179.07 0))
+    (property "Footprint" "" (id 2) (at 43.18 173.99 0)
+      (effects (font (size 1.27 1.27)) hide)
+    )
+    (property "Datasheet" "" (id 3) (at 43.18 173.99 0)
+      (effects (font (size 1.27 1.27)) hide)
+    )
+    (pin "1")
   )
   (symbol (lib_id "Device:C") (at 194.31 46.99 0) (unit 1)
@@
     (pin "1")
   )
+  (symbol (lib_id "Device:C") (at 43.18 170.18 0) (unit 1)
+    (in_bom yes) (on_board yes) (fields_autoplaced)
+    (property "Reference" "C2" (id 0) (at 46.99 168.9099 0)
+      (effects (font (size 1.27 1.27)) (justify left))
+    )
+    (property "Value" "10u" (id 1) (at 46.99 171.4499 0)
+      (effects (font (size 1.27 1.27)) (justify left))
+    )
+    (property "Footprint" "Capacitor_SMD:C_0805_2012Metric_Pad1.18x1.45mm_HandSolder" (id 2) (at 44.1452 173.99 0)
+      (effects (font (size 1.27 1.27)) hide)
+    )
+    (property "Datasheet" "~" (id 3) (at 43.18 170.18 0)
+      (effects (font (size 1.27 1.27)) hide)
+    )
+    (pin "1")
+    (pin "2")
+  )
   (symbol (lib_id "power:GND") (at 233.68 50.8 0) (unit 1)
     (in_bom yes) (on_board yes) (fields_autoplaced)
@@
     (property "Reference" "J4" (id 0) (at 134.62 137.16 0))
     (property "Value" "USB2.0_C" (id 1) (at 134.62 139.7 0))
-    (property "Footprint" "esp32-dev-boards:USB-C-12-Pin-MidMount" (id 2) (at 138.43 160.02 0)
+    (property "Footprint" "esp32-dev-boards:USB-C-12-Pin-MidMount-ali-v4" (id 2) (at 138.43 160.02 0)
       (effects (font (size 1.27 1.27)) hide)
     )
@@
       (reference "#PWR07") (unit 1) (value "GND") (footprint "")
     )
+    (path "/b0b4f256-782a-48ea-b7fd-72843837e4cc"
+      (reference "#PWR08") (unit 1) (value "GND") (footprint "")
+    )
     (path "/55693a61-f125-44cc-b8ca-577b28078d6d"
       (reference "#PWR011") (unit 1) (value "GND") (footprint "")
@@
       (reference "C1") (unit 1) (value "1u") (footprint "Capacitor_SMD:C_0805_2012Metric_Pad1.18x1.45mm_HandSolder")
     )
+    (path "/cd546684-b5d4-453d-a49b-278119e79c29"
+      (reference "C2") (unit 1) (value "10u") (footprint "Capacitor_SMD:C_0805_2012Metric_Pad1.18x1.45mm_HandSolder")
+    )
     (path "/b3013d9b-e7a6-411e-be9a-47f834d8d980"
       (reference "C3") (unit 1) (value "10u") (footprint "Capacitor_SMD:C_0805_2012Metric_Pad1.18x1.45mm_HandSolder")
@@
     )
     (path "/a79ce51b-1c51-458b-929b-aca8897d5bc1"
-      (reference "C5") (unit 1) (value "10u") (footprint "Capacitor_SMD:C_0805_2012Metric_Pad1.18x1.45mm_HandSolder")
+      (reference "C5") (unit 1) (value "100n") (footprint "Capacitor_SMD:C_0805_2012Metric_Pad1.18x1.45mm_HandSolder")
     )
     (path "/98f90266-3d95-4ee7-b973-d123d1ae624b"
-      (reference "C6") (unit 1) (value "100n") (footprint "Capacitor_SMD:C_0805_2012Metric_Pad1.18x1.45mm_HandSolder")
+      (reference "C6") (unit 1) (value "10u") (footprint "Capacitor_SMD:C_0805_2012Metric_Pad1.18x1.45mm_HandSolder")
     )
     (path "/31517704-09dc-470d-aaec-ee756808534f"
@@
     )
     (path "/e3b43fdb-6eb5-4f00-ba13-582445a8931a"
-      (reference "J4") (unit 1) (value "USB2.0_C") (footprint "esp32-dev-boards:USB-C-12-Pin-MidMount")
+      (reference "J4") (unit 1) (value "USB2.0_C") (footprint "esp32-dev-boards:USB-C-12-Pin-MidMount-ali-v4")
     )
     (path "/89502c1e-cb15-4216-b258-c3c5ffbaefc8"

Commit message: before routing
Parts:
- removed C4: 100n, Capacitor_SMD:C_0805_2012Metric_Pad1.18x1.45mm_HandSolder, symbol Device:C
- removed C6: 10u, Capacitor_SMD:C_0805_2012Metric_Pad1.18x1.45mm_HandSolder, symbol Device:C
- removed J1: ESP32-C3-DEVKITM-1-J1, esp32-dev-boards:ESP32-C3-DEVKITM-J1, symbol esp32-dev-boards:ESP32-C3-DEVKITM-1-J1
- removed J2: ESP32-C3-DEVKITM-1-J2, esp32-dev-boards:ESP32-C3-DEVKITM-J2, symbol esp32-dev-boards:ESP32-C3-DEVKITM-1-J2
- added C7: 100n, $74th:Capacitor_0805_2012, symbol Device:C
- added CH2: ProMicro-RightPin, $74th:ProMicro_LIKE_RIGHT, symbol $74th:ProMicro-RightPin
- added CH3: ProMicro-LeftPin, $74th:ProMicro_LIKE_LEFT, symbol $74th:ProMicro-LeftPin
- added R5, R6: 0, $74th:Register_0805_2012, symbol Device:R
- added R8: 10k, $74th:Register_0805_2012, symbol Device:R
- C1: value 1u -> 100n; footprint Capacitor_SMD:C_0805_2012Metric_Pad1.18x1.45mm_HandSolder -> $74th:Capacitor_0805_2012
- C2, C3, C5: footprint Capacitor_SMD:C_0805_2012Metric_Pad1.18x1.45mm_HandSolder -> $74th:Capacitor_0805_2012
- D5: footprint LED_SMD:LED_0805_2012Metric_Pad1.15x1.40mm_HandSolder -> $74th:LED_0805_2012Metric_Pad1.15x1.40mm_HandSolder
- J3: footprint esp32-dev-boards:BoxPinHeader_2x03_P1.27mm_Vertical -> $74th:BoxPinHeader_2x03_P1.27mm_Vertical
- J4: footprint esp32-dev-boards:USB-C-12-Pin-MidMount-ali-v4 -> $74th:USB-C-12-Pin-SMD
- R1, R2, R3, R4: footprint Resistor_SMD:R_0805_2012Metric_Pad1.20x1.40mm_HandSolder -> $74th:Register_0805_2012
- SW1, SW2: footprint esp32-dev-boards:SKRPABE010 -> $74th:SKRPABE010
- U1: footprint Espressif:ESP32-C3-MINI-1_Hand-Soldering -> Espressif:ESP32-C3-MINI-1
- U2: footprint Package_TO_SOT_SMD:SOT-223-3_TabPin2 -> $74th:Regulator_AMS1117_SOT-89
Connections:
- net +3V3: now also R3.2, CH2.9 (3V3), R8.2
- net +5V: now also CH2.12 (RAW); no longer R3.2
- net CHIP_PU: now also CH2.10 (~{RESET}); no longer C1.1, R1.1, SW2.2, U1.8 (EN/CHIP_PU)
- net GND: now also C7.2, CH2.1 (10/A10), CH2.11 (GND), CH3.11 (8/A8), CH3.12 (9/A9), CH3.3 (GND), CH3.4 (GND)
- net GPIO0: now also CH3.6 (3/SCL); no longer SW1.2
- net GPIO1: now also CH3.5 (2/SDA)
- net GPIO10: now also CH3.8 (5)
- net GPIO18: now also CH3.9 (6/A7), R5.1; no longer J4.2 (D-)
- net GPIO19: now also CH3.10 (7), R6.1; no longer J4.3 (D+)
- net GPIO2: now also CH2.5 (18/A0)
- net GPIO3: now also CH2.6 (19/A1)
- net GPIO4: now also CH2.7 (20/A2)
- net GPIO5: now also CH2.8 (21/A3)
- net GPIO6: now also CH2.2 (16/SPI_MOSI)
- net GPIO7: now also CH2.3 (14/SPI_MISO)
- net GPIO8: now also CH3.7 (4/A6), R8.1
- net GPIO9: now also SW1.2, C7.1, CH2.4 (15/SPI_SCK)
- net U0RXD: now also CH3.2 (0/RX)
- net U0TXD: now also CH3.1 (1/TX)
- new net: C1.1, R1.1, SW2.2, U1.8 (EN/CHIP_PU)
- new net: J4.3 (D+), R6.2
- new net: J4.2 (D-), R5.2
Other:
- moved on the sheet: C1, C2, C3, D5, J3, J4, R1, R2, R3, R4, SW1, SW2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

Commit message: uo
Connections:
- net GND: now also U1.37 (GND), U1.38 (GND), U1.39 (GND), U1.40 (GND), U1.41 (GND), U1.42 (GND), U1.43 (GND), U1.44 (GND), U1.45 (GND), U1.46 (GND), U1.47 (GND), U1.48 (GND), U1.49 (GND), U1.50 (GND), U1.51 (GND), U1.52 (GND), U1.53 (GND); no longer C2.2
Other:
- moved on the sheet: C1, C2, C7, R1, R8, SW1, SW2

Commit message: before panelize
Parts:
- renumbered C2 to C1, C7 to C2, C1 to C3, C5 to C4, C3 to C5, CH3 to CH1, D5 to D1, J3 to J1, J4 to J2, R8 to R2, R6 to R3, R5 to R4, R3 to R5, R2 to R6, R4 to R7, SW2 to SW1, SW1 to SW2
Changed lines of the file:
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@@
   (symbol (lib_id "Device:R") (at 208.28 147.32 180) (unit 1)
     (in_bom yes) (on_board yes) (dnp no) (fields_autoplaced)
-    (property "Reference" "R2" (at 210.82 146.0499 0)
+    (property "Reference" "R6" (at 210.82 146.0499 0)
       (effects (font (size 1.27 1.27)) (justify right))
     )
@@
       (project "ESP32-C3-MINI-1"
         (path "/1f0126c3-e865-4b7c-bf68-4d53d0d38c5a"
-          (reference "R2") (unit 1)
+          (reference "R6") (unit 1)
         )
       )
@@
   (symbol (lib_id "Switch:SW_Push") (at 44.45 119.38 90) (unit 1)
     (in_bom yes) (on_board yes) (dnp no) (fields_autoplaced)
-    (property "Reference" "SW2" (at 45.72 118.745 90)
+    (property "Reference" "SW1" (at 45.72 118.745 90)
       (effects (font (size 1.27 1.27)) (justify right))
     )
@@
       (project "ESP32-C3-MINI-1"
         (path "/1f0126c3-e865-4b7c-bf68-4d53d0d38c5a"
-          (reference "SW2") (unit 1)
+          (reference "SW1") (unit 1)
         )
       )
@@
   (symbol (lib_id "Device:LED") (at 245.11 54.61 90) (unit 1)
     (in_bom yes) (on_board yes) (dnp no) (fields_autoplaced)
-    (property "Reference" "D5" (at 248.92 54.9274 90)
+    (property "Reference" "D1" (at 248.92 54.9274 90)
       (effects (font (size 1.27 1.27)) (justify right))
     )
@@
       (project "ESP32-C3-MINI-1"
         (path "/1f0126c3-e865-4b7c-bf68-4d53d0d38c5a"
-          (reference "D5") (unit 1)
+          (reference "D1") (unit 1)
         )
       )
@@
   (symbol (lib_id "Switch:SW_Push") (at 135.89 162.56 90) (unit 1)
     (in_bom yes) (on_board yes) (dnp no) (fields_autoplaced)
-    (property "Reference" "SW1" (at 137.16 161.925 90)
+    (property "Reference" "SW2" (at 137.16 161.925 90)
       (effects (font (size 1.27 1.27)) (justify right))
     )
@@
       (project "ESP32-C3-MINI-1"
         (path "/1f0126c3-e865-4b7c-bf68-4d53d0d38c5a"
-          (reference "SW1") (unit 1)
+          (reference "SW2") (unit 1)
         )
       )
@@
   (symbol (lib_id "Device:R") (at 217.17 147.32 180) (unit 1)
     (in_bom yes) (on_board yes) (dnp no) (fields_autoplaced)
-    (property "Reference" "R4" (at 219.71 146.0499 0)
+    (property "Reference" "R7" (at 219.71 146.0499 0)
       (effects (font (size 1.27 1.27)) (justify right))
     )
@@
       (project "ESP32-C3-MINI-1"
         (path "/1f0126c3-e865-4b7c-bf68-4d53d0d38c5a"
-          (reference "R4") (unit 1)
+          (reference "R7") (unit 1)
         )
       )
@@
   (symbol (lib_id "Device:R") (at 218.44 129.54 270) (unit 1)
     (in_bom yes) (on_board yes) (dnp no)
-    (property "Reference" "R6" (at 218.44 124.46 90)
+    (property "Reference" "R3" (at 218.44 124.46 90)
       (effects (font (size 1.27 1.27)))
     )
@@
       (project "ESP32-C3-MINI-1"
         (path "/1f0126c3-e865-4b7c-bf68-4d53d0d38c5a"
-          (reference "R6") (unit 1)
+          (reference "R3") (unit 1)
         )
       )
@@
   (symbol (lib_id "esp32-dev-boards:ESPProg-UART") (at 129.54 41.91 0) (unit 1)
     (in_bom yes) (on_board yes) (dnp no) (fields_autoplaced)
-    (property "Reference" "J3" (at 129.54 36.83 0)
+    (property "Reference" "J1" (at 129.54 36.83 0)
       (effects (font (size 1.27 1.27)))
     )
@@
       (project "ESP32-C3-MINI-1"
         (path "/1f0126c3-e865-4b7c-bf68-4d53d0d38c5a"
-          (reference "J3") (unit 1)
+          (reference "J1") (unit 1)
         )
       )
@@
   (symbol (lib_id "Device:C") (at 233.68 46.99 0) (unit 1)
     (in_bom yes) (on_board yes) (dnp no) (fields_autoplaced)
-    (property "Reference" "C5" (at 237.49 45.7199 0)
+    (property "Reference" "C4" (at 237.49 45.7199 0)
       (effects (font (size 1.27 1.27)) (justify left))
     )
@@
       (project "ESP32-C3-MINI-1"
         (path "/1f0126c3-e865-4b7c-bf68-4d53d0d38c5a"
-          (reference "C5") (unit 1)
+          (reference "C4") (unit 1)
         )
       )
@@
   (symbol (lib_id "Device:C") (at 31.75 119.38 0) (unit 1)
     (in_bom yes) (on_board yes) (dnp no) (fields_autoplaced)
-    (property "Reference" "C1" (at 35.56 118.745 0)
+    (property "Reference" "C3" (at 35.56 118.745 0)
       (effects (font (size 1.27 1.27)) (justify left))
     )
@@
       (project "ESP32-C3-MINI-1"
         (path "/1f0126c3-e865-4b7c-bf68-4d53d0d38c5a"
-          (reference "C1") (unit 1)
+          (reference "C3") (unit 1)
         )
       )
@@
   (symbol (lib_id "Device:R") (at 218.44 121.92 270) (unit 1)
     (in_bom yes) (on_board yes) (dnp no) (fields_autoplaced)
-    (property "Reference" "R5" (at 218.44 116.84 90)
+    (property "Reference" "R4" (at 218.44 116.84 90)
       (effects (font (size 1.27 1.27)))
     )
@@
       (project "ESP32-C3-MINI-1"
         (path "/1f0126c3-e865-4b7c-bf68-4d53d0d38c5a"
+          (reference "R4") (unit 1)
+        )
+      )
+    )
+  )
+  (symbol (lib_id "Device:R") (at 245.11 46.99 180) (unit 1)
+    (in_bom yes) (on_board yes) (dnp no) (fields_autoplaced)
+    (property "Reference" "R5" (at 247.65 45.7199 0)
+      (effects (font (size 1.27 1.27)) (justify right))
+    )
+    (property "Value" "1k" (at 247.65 48.2599 0)
+      (effects (font (size 1.27 1.27)) (justify right))
+    )
+    (property "Footprint" "$74th:Register_0805_2012" (at 246.888 46.99 90)
+      (effects (font (size 1.27 1.27)) hide)
+    )
+    (property "Datasheet" "~" (at 245.11 46.99 0)
+      (effects (font (size 1.27 1.27)) hide)
+    )
+    (pin "1")
+    (pin "2")
+    (instances
+      (project "ESP32-C3-MINI-1"
+        (path "/1f0126c3-e865-4b7c-bf68-4d53d0d38c5a"
           (reference "R5") (unit 1)
         )
@@
     )
   )
-  (symbol (lib_id "Device:R") (at 245.11 46.99 180) (unit 1)
-    (in_bom yes) (on_board yes) (dnp no) (fields_autoplaced)
-    (property "Reference" "R3" (at 247.65 45.7199 0)
-      (effects (font (size 1.27 1.27)) (justify right))
-    )
-    (property "Value" "1k" (at 247.65 48.2599 0)
-      (effects (font (size 1.27 1.27)) (justify right))
-    )
-    (property "Footprint" "$74th:Register_0805_2012" (at 246.888 46.99 90)
-      (effects (font (size 1.27 1.27)) hide)
-    )
-    (property "Datasheet" "~" (at 245.11 46.99 0)
-      (effects (font (size 1.27 1.27)) hide)
-    )
-    (pin "1")
-    (pin "2")
-    (instances
-      (project "ESP32-C3-MINI-1"
-        (path "/1f0126c3-e865-4b7c-bf68-4d53d0d38c5a"
-          (reference "R3") (unit 1)
-        )
-      )
-    )
-  )
   (symbol (lib_id "power:GND") (at 83.82 106.68 0) (unit 1)
     (in_bom yes) (on_board yes) (dnp no) (fields_autoplaced)
@@
   (symbol (lib_id "Device:R") (at 135.89 151.13 180) (unit 1)
     (in_bom yes) (on_board yes) (dnp no) (fields_autoplaced)
-    (property "Reference" "R8" (at 138.43 149.8599 0)
+    (property "Reference" "R2" (at 138.43 149.8599 0)
       (effects (font (size 1.27 1.27)) (justify right))
     )
@@
       (project "ESP32-C3-MINI-1"
         (path "/1f0126c3-e865-4b7c-bf68-4d53d0d38c5a"
-          (reference "R8") (unit 1)
+          (reference "R2") (unit 1)
         )
       )
@@
   (symbol (lib_id "Device:C") (at 200.66 46.99 0) (unit 1)
     (in_bom yes) (on_board yes) (dnp no) (fields_autoplaced)
-    (property "Reference" "C3" (at 204.47 45.7199 0)
+    (property "Reference" "C5" (at 204.47 45.7199 0)
       (effects (font (size 1.27 1.27)) (justify left))
     )
@@
       (project "ESP32-C3-MINI-1"
         (path "/1f0126c3-e865-4b7c-bf68-4d53d0d38c5a"
-          (reference "C3") (unit 1)
+          (reference "C5") (unit 1)
         )
       )
@@
   (symbol (lib_id "Device:C") (at 144.78 161.29 0) (unit 1)
     (in_bom yes) (on_board yes) (dnp no) (fields_autoplaced)
-    (property "Reference" "C7" (at 148.59 160.655 0)
+    (property "Reference" "C2" (at 148.59 160.655 0)
       (effects (font (size 1.27 1.27)) (justify left))
     )
@@
       (project "ESP32-C3-MINI-1"
         (path "/1f0126c3-e865-4b7c-bf68-4d53d0d38c5a"
-          (reference "C7") (unit 1)
+          (reference "C2") (unit 1)
         )
       )
@@
   (symbol (lib_id "Device:C") (at 83.82 104.14 0) (unit 1)
     (in_bom yes) (on_board yes) (dnp no) (fields_autoplaced)
-    (property "Reference" "C2" (at 87.63 102.8699 0)
+    (property "Reference" "C1" (at 87.63 102.8699 0)
       (effects (font (size 1.27 1.27)) (justify left))
     )
@@
       (project "ESP32-C3-MINI-1"
         (path "/1f0126c3-e865-4b7c-bf68-4d53d0d38c5a"
-          (reference "C2") (unit 1)
+          (reference "C1") (unit 1)
         )
       )
@@
   (symbol (lib_id "$74th:ProMicro-LeftPin") (at 45.72 50.8 0) (unit 1)
     (in_bom yes) (on_board yes) (dnp no)
-    (property "Reference" "CH3" (at 44.45 35.56 0)
+    (property "Reference" "CH1" (at 44.45 35.56 0)
       (effects (font (size 1.27 1.27)) (justify left))
     )
@@
       (project "ESP32-C3-MINI-1"
         (path "/1f0126c3-e865-4b7c-bf68-4d53d0d38c5a"
-          (reference "CH3") (unit 1)
+          (reference "CH1") (unit 1)
         )
       )
@@
   (symbol (lib_id "esp32-dev-boards:USB2.0_C") (at 189.23 134.62 0) (unit 1)
     (in_bom yes) (on_board yes) (dnp no) (fields_autoplaced)
-    (property "Reference" "J4" (at 189.23 111.76 0)
+    (property "Reference" "J2" (at 189.23 111.76 0)
       (effects (font (size 1.27 1.27)))
     )
@@
       (project "ESP32-C3-MINI-1"
         (path "/1f0126c3-e865-4b7c-bf68-4d53d0d38c5a"
-          (reference "J4") (unit 1)
-        )
-      )
+          (reference "J2") (unit 1)
+        )
+      )
