File: ESP32-C3-MINI-1/ESP32-C3-MINI-1-panelized.kicad_pcb (KiCad board)
At the start: 2 copper layers, 73 x 52 mm, 165 parts, among them J1 ESP32-C3-DEVKITM-1-J2, J2 ESP32-C3-DEVKITM-1-J1, J3 UART, J4 ESP32-C3-DEVKITM-1-J2, J5 ESP32-C3-DEVKITM-1-J1, J6 UART, J7 ESP32-C3-DEVKITM-1-J2, J8 ESP32-C3-DEVKITM-1-J1, J9 UART, SW1 RESET, SW2 BOOT, SW3 BOOT, SW4 RESET, SW5 BOOT, SW6 RESET, U1 ESP32-C3-MINI-1, U2 AMS1117-3.3, U3 ESP32-C3-MINI-1, U4 AMS1117-3.3, U5 ESP32-C3-MINI-1, U6 AMS1117-3.3

Commit message: before panelize
Parts:
- removed C10, C11, C13: 10u, Capacitor_SMD:C_0805_2012Metric_Pad1.18x1.45mm_HandSolder
- removed C12, C15, C4, C6, C9: 100n, Capacitor_SMD:C_0805_2012Metric_Pad1.18x1.45mm_HandSolder
- removed C14, C8: 1u, Capacitor_SMD:C_0805_2012Metric_Pad1.18x1.45mm_HandSolder
- removed D1, D2, D3: PWR, LED_SMD:LED_0805_2012Metric_Pad1.15x1.40mm_HandSolder
- removed J1, J7: ESP32-C3-DEVKITM-1-J2, esp32-dev-boards:ESP32-C3-DEVKITM-J2
- removed J2, J5, J8: ESP32-C3-DEVKITM-1-J1, esp32-dev-boards:ESP32-C3-DEVKITM-J1
- removed J6, J9: UART, esp32-dev-boards:UART
- removed the REF** at (27.7, 63.0)
- removed the REF** at (53.0, 63.0)
- removed the REF** at (61.6, 29.5)
- removed the REF** at (84.0, 17.0)
- removed the REF** at (84.0, 51.5)
- removed the REF** at (73.3, 19.0)
- removed the REF** at (17.0, 63.0)
- removed the REF** at (63.6, 29.5)
- removed the REF** at (39.3, 42.5)
- removed the REF** at (39.3, 39.5)
- removed the REF** at (39.3, 31.5)
- removed the REF** at (84.0, 41.5)
- removed the REF** at (16.0, 19.0)
- removed the REF** at (61.6, 50.5)
- removed the REF** at (16.0, 63.0)
- removed the REF** at (19.0, 28.5)
- removed the REF** at (41.3, 28.5)
- removed the REF** at (63.6, 39.5)
- removed the REF** at (17.0, 19.0)
- removed the REF** at (63.6, 50.5)
- removed the REF** at (84.0, 52.5)
- removed the REF** at (61.6, 42.5)
- removed the REF** at (87.0, 19.0)
- removed the REF** at (84.0, 50.5)
- removed the REF** at (61.6, 30.5)
- removed the REF** at (61.6, 52.5)
- removed the REF** at (19.0, 31.5)
- removed the REF** at (84.0, 65.0)
- removed the REF** at (63.6, 30.5)
- removed the REF** at (19.0, 53.5)
- removed the REF** at (88.0, 63.0)
- removed the REF** at (39.3, 53.5)
- removed the REF** at (63.6, 31.5)
- removed the REF** at (75.3, 63.0)
- removed the REF** at (61.6, 40.5)
- removed the REF** at (41.3, 52.5)
- removed the REF** at (30.7, 63.0)
- removed the REF** at (19.0, 40.5)
- removed the REF** at (39.3, 30.5)
- removed the REF** at (41.3, 31.5)
- removed the REF** at (39.3, 52.5)
- removed the REF** at (19.0, 50.5)
- removed the REF** at (75.3, 19.0)
- removed the REF** at (39.3, 41.5)
- removed the REF** at (51.0, 63.0)
- removed the REF** at (19.0, 39.5)
- removed the REF** at (19.0, 29.5)
- removed the REF** at (61.6, 31.5)
- removed the REF** at (72.3, 19.0)
- removed the REF** at (30.7, 19.0)
- removed the REF** at (39.3, 28.5)
- removed the REF** at (72.3, 63.0)
- removed the REF** at (84.0, 66.0)
- removed the REF** at (84.0, 15.0)
- removed the REF** at (63.6, 28.5)
- removed the REF** at (19.0, 15.0)
- removed the REF** at (63.6, 51.5)
- removed the REF** at (29.7, 19.0)
- removed the REF** at (63.6, 42.5)
- removed the REF** at (50.0, 19.0)
- removed the REF** at (61.6, 51.5)
- removed the REF** at (39.3, 51.5)
- removed the REF** at (41.3, 53.5)
- removed the REF** at (86.0, 19.0)
- removed the REF** at (63.6, 53.5)
- removed the REF** at (84.0, 39.5)
- removed the REF** at (61.6, 28.5)
- removed the REF** at (63.6, 40.5)
- removed the REF** at (19.0, 16.0)
- removed the REF** at (41.3, 39.5)
- removed the REF** at (84.0, 53.5)
- removed the REF** at (28.7, 63.0)
- removed the REF** at (41.3, 41.5)
- removed the REF** at (41.3, 40.5)
- removed the REF** at (61.6, 41.5)
- removed the REF** at (19.0, 30.5)
- removed the REF** at (19.0, 17.0)
- removed the REF** at (73.3, 63.0)
- removed the REF** at (63.6, 41.5)
- removed the REF** at (41.3, 30.5)
- removed the REF** at (84.0, 67.0)
- removed the REF** at (19.0, 51.5)
- removed the REF** at (84.0, 30.5)
- removed the REF** at (19.0, 67.0)
- removed the REF** at (84.0, 28.5)
- removed the REF** at (29.7, 63.0)
- removed the REF** at (52.0, 19.0)
- removed the REF** at (19.0, 66.0)
- removed the REF** at (84.0, 16.0)
- removed the REF** at (41.3, 51.5)
- removed the REF** at (41.3, 50.5)
- removed the REF** at (19.0, 65.0)
- removed the REF** at (53.0, 19.0)
- removed the REF** at (51.0, 19.0)
- removed the REF** at (87.0, 63.0)
- removed the REF** at (41.3, 42.5)
- removed the REF** at (15.0, 63.0)
- removed the REF** at (84.0, 29.5)
- removed the REF** at (74.3, 19.0)
- removed the REF** at (84.0, 31.5)
- removed the REF** at (74.3, 63.0)
- removed the REF** at (84.0, 40.5)
- removed the REF** at (41.3, 29.5)
- removed the REF** at (63.6, 52.5)
- removed the REF** at (28.7, 19.0)
- removed the REF** at (39.3, 40.5)
- removed the REF** at (84.0, 42.5)
- removed the REF** at (50.0, 63.0)
- removed the REF** at (61.6, 39.5)
- removed the REF** at (19.0, 52.5)
- removed the REF** at (88.0, 19.0)
- removed the REF** at (52.0, 63.0)
- removed the REF** at (19.0, 42.5)
- removed the REF** at (39.3, 50.5)
- removed the REF** at (61.6, 53.5)
- removed the REF** at (15.0, 19.0)
- removed the REF** at (86.0, 63.0)
- removed the REF** at (19.0, 41.5)
- removed the REF** at (39.3, 29.5)
- removed the REF** at (27.7, 19.0)
- removed SW3, SW5: BOOT, esp32-dev-boards:SKRPABE010
- removed SW4, SW6: RESET, esp32-dev-boards:SKRPABE010
- removed U3, U5: ESP32-C3-MINI-1, esp32-dev-boards:ESP32-C3-MINI-1
- removed U4, U6: AMS1117-3.3, Package_TO_SOT_SMD:SOT-223-3_TabPin2
- added CH2: ProMicro-RightPin, $74th:ProMicro_LIKE_RIGHT, F.Cu at (108.0, 100.3)
- added CH3: ProMicro-LeftPin, $74th:ProMicro_LIKE_LEFT, F.Cu at (90.2, 99.1)
- added D5: PWR, $74th:LED_0805_2012Metric_Pad1.15x1.40mm_HandSolder, F.Cu at (105.2, 112.0)
- added R8: 10k, $74th:Register_0805_2012, B.Cu at (99.1, 94.7)
- added REF**: JLCJLCJLCJLC, $74th:JLCJLCJLCJLC, F.Cu at (97.9, 86.7)
- C1, C7: value 10u -> 100n; footprint Capacitor_SMD:C_0805_2012Metric_Pad1.18x1.45mm_HandSolder -> $74th:Capacitor_0805_2012; moved to B.Cu
- C2: footprint Capacitor_SMD:C_0805_2012Metric_Pad1.18x1.45mm_HandSolder -> $74th:Capacitor_0805_2012; moved to B.Cu
- C3: value 100n -> 10u; footprint Capacitor_SMD:C_0805_2012Metric_Pad1.18x1.45mm_HandSolder -> $74th:Capacitor_0805_2012; moved to B.Cu
- C5: value 1u -> 100n; footprint Capacitor_SMD:C_0805_2012Metric_Pad1.18x1.45mm_HandSolder -> $74th:Capacitor_0805_2012; moved to B.Cu
- J3: value UART -> ESPProg-UART; footprint esp32-dev-boards:UART -> $74th:BoxPinHeader_2x03_P1.27mm_Vertical
- J4: value ESP32-C3-DEVKITM-1-J2 -> USB2.0_C; footprint esp32-dev-boards:ESP32-C3-DEVKITM-J2 -> $74th:USB-C-12-Pin-SMD
- R1: value 5.1k -> 10k; footprint Resistor_SMD:R_0805_2012Metric_Pad1.20x1.40mm_HandSolder -> $74th:Register_0805_2012; moved to B.Cu
- R2: value 10k -> 5.1k; footprint Resistor_SMD:R_0805_2012Metric_Pad1.20x1.40mm_HandSolder -> $74th:Register_0805_2012; moved to B.Cu
- R3: value 10k -> 1k; footprint Resistor_SMD:R_0805_2012Metric_Pad1.20x1.40mm_HandSolder -> $74th:Register_0805_2012; moved to B.Cu
- R4: footprint Resistor_SMD:R_0805_2012Metric_Pad1.20x1.40mm_HandSolder -> $74th:Register_0805_2012; moved to B.Cu
- R5: value 10k -> 0; footprint Resistor_SMD:R_0805_2012Metric_Pad1.20x1.40mm_HandSolder -> $74th:Register_0805_2012; moved to B.Cu
- R6: value 5.1k -> 0; footprint Resistor_SMD:R_0805_2012Metric_Pad1.20x1.40mm_HandSolder -> $74th:Register_0805_2012; moved to B.Cu
- SW1: value RESET -> BOOT; footprint esp32-dev-boards:SKRPABE010 -> $74th:SKRPABE010
- SW2: value BOOT -> RESET; footprint esp32-dev-boards:SKRPABE010 -> $74th:SKRPABE010
- U1: footprint esp32-dev-boards:ESP32-C3-MINI-1 -> Espressif:ESP32-C3-MINI-1
- U2: footprint Package_TO_SOT_SMD:SOT-223-3_TabPin2 -> $74th:Regulator_AMS1117_SOT-89; moved to B.Cu
- moved J4 96.9 mm to (99.1, 113.2)
- moved U2 96.2 mm to (103.5, 103.5), turned to 90 degrees
- moved R2 95.9 mm to (101.3, 112.0), turned to 90 degrees
- moved C3 92.8 mm to (100.0, 108.8)
- moved U1 90.0 mm to (99.0, 86.9)
- moved C1 88.6 mm to (95.8, 92.7), turned to 0 degrees
- moved SW1 87.1 mm to (102.2, 97.8)
- moved J3 86.6 mm to (97.2, 102.9), turned to 90 degrees
- moved C5 86.0 mm to (102.6, 98.6), turned to 180 degrees
- moved R4 81.0 mm to (96.8, 112.0)
- moved R3 80.8 mm to (105.2, 110.0), turned to 90 degrees
- moved C2 80.3 mm to (96.1, 86.9)
- moved R1 79.1 mm to (95.8, 90.7), turned to 180 degrees
- moved SW2 76.4 mm to (95.5, 97.8)
- moved C7 73.8 mm to (99.3, 91.7), turned to 90 degrees
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Connections:
- C1 pad 1: Board_0-+3V3 -> Net-(U1-EN/CHIP_PU)
- C1 pad 2: Board_0-GND -> GND
- C2 pad 1: Board_0-+5V -> +3V3
- C2 pad 2: Board_0-GND -> unconnected-(C2-Pad2)
- C3 pad 1: Board_0-+5V -> +5V
- C3 pad 2: Board_0-GND -> GND
- C5 pad 1: Board_0-CHIP_PU -> +3V3
- C5 pad 2: Board_0-GND -> GND
- C7 pad 1: Board_1-+3V3 -> GPIO9
- C7 pad 2: Board_1-GND -> GND
- J3 pad 1: Board_0-U0TXD -> CHIP_PU
- J3 pad 2: Board_0-U0RXD -> +5V
- J3 pad 3: Board_0-+5V -> U0TXD
- J3 pad 4: Board_0-GND -> GND
- J3 pad 5: Board_0-CHIP_PU -> U0RXD
- J3 pad 6: Board_0-GPIO0 -> GPIO0
- J4 pad 1: Board_1-GND -> +5V
- J4 pad 2: Board_1-U0TXD -> Net-(J4-D-)
- J4 pad 3: Board_1-U0RXD -> Net-(J4-D+)
- J4 pad 4: Board_1-GND -> GND
- J4 pad 5: Board_1-GPIO9 -> Net-(J4-CC1)
- J4 pad 6: Board_1-GPIO8 -> Net-(J4-CC2)
- R1 pad 1: Board_0-Net-(D5-Pad2) -> Net-(U1-EN/CHIP_PU)
- R1 pad 2: Board_0-+3V3 -> +3V3
- R2 pad 1: Board_0-CHIP_PU -> GND
- R2 pad 2: Board_0-+3V3 -> Net-(J4-CC2)
- R3 pad 1: Board_1-CHIP_PU -> Net-(D5-A)
- R3 pad 2: Board_1-+3V3 -> +3V3
- R4 pad 1: Board_1-Net-(D5-Pad2) -> GND
- R4 pad 2: Board_1-+3V3 -> Net-(J4-CC1)
- R5 pad 1: Board_2-CHIP_PU -> GPIO18
- R5 pad 2: Board_2-+3V3 -> Net-(J4-D-)
- R6 pad 1: Board_2-Net-(D5-Pad2) -> GPIO19
- R6 pad 2: Board_2-+3V3 -> Net-(J4-D+)
- SW1 pad 1: Board_0-GND -> GND
- SW1 pad 2: Board_0-CHIP_PU -> GPIO9
- SW2 pad 1: Board_0-GND -> GND
- SW2 pad 2: Board_0-GPIO0 -> Net-(U1-EN/CHIP_PU)
- U1 pad 1: Board_0-GND -> GND
- U1 pad 11: Board_0-GND -> GND
- U1 pad 12: Board_0-GPIO0 -> GPIO0
- U1 pad 13: Board_0-GPIO1 -> GPIO1
- U1 pad 14: Board_0-GND -> GND
- U1 pad 16: Board_0-GPIO10 -> GPIO10
- U1 pad 18: Board_0-GPIO4 -> GPIO4
- U1 pad 19: Board_0-GPIO5 -> GPIO5
- U1 pad 2: Board_0-GND -> GND
- U1 pad 20: Board_0-GPIO6 -> GPIO6
- U1 pad 21: Board_0-GPIO7 -> GPIO7
- U1 pad 22: Board_0-GPIO8 -> GPIO8
- U1 pad 23: Board_0-GPIO9 -> GPIO9
- U1 pad 26: Board_0-GPIO18 -> GPIO18
- U1 pad 27: Board_0-GPIO19 -> GPIO19
- U1 pad 3: Board_0-+3V3 -> +3V3
- U1 pad 30: Board_0-U0RXD -> U0RXD
- U1 pad 31: Board_0-U0TXD -> U0TXD
- U1 pad 36: Board_0-GND -> GND
- U1 pad 5: Board_0-GPIO2 -> GPIO2
- U1 pad 6: Board_0-GPIO3 -> GPIO3
- U1 pad 8: Board_0-CHIP_PU -> Net-(U1-EN/CHIP_PU)
- U2 pad 1: Board_0-GND -> GND
- U2 pad 2: Board_0-+3V3 -> +3V3
- U2 pad 3: Board_0-+5V -> +5V
Routing:
- net GND: track 0.00 -> 63.6 mm, vias 0 -> 26
- net +3V3: track 0.00 -> 57.5 mm, vias 0 -> 1
- net +5V: track 0.00 -> 57.1 mm, vias 0 -> 3
- net Board_1-+3V3: track 55.1 -> 0.00 mm
- net Board_0-+3V3: track 55.1 -> 0.00 mm
- net Board_2-+3V3: track 55.1 -> 0.00 mm
- net Board_2-CHIP_PU: track 47.5 -> 0.00 mm, vias 1 -> 0
- net Board_1-CHIP_PU: track 47.5 -> 0.00 mm, vias 1 -> 0
- net Board_0-CHIP_PU: track 47.5 -> 0.00 mm, vias 1 -> 0
- net Board_0-U0TXD: track 47.0 -> 0.00 mm
- net Board_2-U0TXD: track 47.0 -> 0.00 mm
- net Board_1-U0TXD: track 47.0 -> 0.00 mm
- net Board_2-GPIO0: track 46.2 -> 0.00 mm, vias 1 -> 0
- net Board_1-GPIO0: track 46.2 -> 0.00 mm, vias 1 -> 0
- net Board_0-GPIO0: track 46.2 -> 0.00 mm, vias 1 -> 0
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- added copper zone on B.Cu, net GND
- added copper zone on F.Cu, net GND
- removed copper zone on B.Cu, net Board_0-GND
- removed copper zone on F.Cu, net Board_0-GND
- removed copper zone on B.Cu, net Board_1-GND
- removed copper zone on F.Cu, net Board_1-GND
- removed copper zone on B.Cu, net Board_2-GND
- removed copper zone on F.Cu, net Board_2-GND
Other:
- board size 73 x 52 mm -> 20.3 x 31.1 mm
- board text added: "0"
- board text added: "3V"
- board text added: "BOOT"
- board text added: "EN"
- board text added: "ESP32C3 DevBoardM"
- board text added: "G"
- board text added: "v1.1.0"
- board text removed: "3V3"
- board text removed: "BT"
- board text removed: "GND"

Commit message: v1.2.0
Parts:
- added G***: LOGO, $74th:74th-4mm, F.Cu at (94.9, 106.8)
- added G***: LOGO, $74th:74th-4mm, B.Cu at (93.4, 104.2)
- added REF**: twitter, $74th:twitter, B.Cu at (94.8, 106.9)
- renumbered C2 to C1, C7 to C2, C1 to C3, C5 to C4, C3 to C5, CH3 to CH1, D5 to D1, J3 to J1, J4 to J2, R8 to R2, R6 to R3, R5 to R4, R3 to R5, R2 to R6, R4 to R7, SW2 to SW1, SW1 to SW2
Routing:
- net GND: track 63.6 -> 66.8 mm
- net U0RXD: track 43.2 -> 44.2 mm
- net Net-(J4-D+): track 11.4 -> 12.2 mm
- net GPIO19: track 43.8 -> 43.2 mm
Other:
- board text added: "ESP32C3"
- board text added: "Micro"
- board text added: "v1.2.0"
