File: ESP32-C3-WROOM-02/ESP32-C3-WROOM-02.kicad_pcb (KiCad board)
At the start: 2 copper layers, 25.4 x 38.1 mm, 20 parts, among them J1 ESP32-C3-DEVKITC-02-J1, J2 ESP32-C3-DEVKITC-02-J2, J3 ESPProg-UART, J4 USB2.0_C, SW1 SW_Push, SW2 SW_Push, U1 AMS1117-3.3, U2 ESP32-C3-WROOM-02

Commit message: up
Parts:
- added REF**: JLCJLCJLCJLC, $74th:JLCJLCJLCJLC, F.Cu at (86.1, 51.4)

Commit message: up
Parts:
- added R5: 10k, esp32-dev-board:Register_0805_2012, B.Cu at (78.1, 57.9)
Routing:
- net +3V3: track 44.8 -> 46.9 mm
- net GPIO8: track 22.7 -> 24.2 mm
- net GPIO9: track 49.3 -> 50.2 mm
Other:
- board text added: "v1.1.0"
- board text removed: "v1.0.0"
