File: ESP32-C3-WROOM-02/ESP32-C3-WROOM-02.kicad_sch (KiCad schematic)
At the start: 20 parts, among them J1 ESP32-C3-DEVKITC-02-J1, J2 ESP32-C3-DEVKITC-02-J2, J3 ESPProg-UART, J4 USB2.0_C, SW1 SW_Push, SW2 SW_Push, U1 AMS1117-3.3, U2 ESP32-C3-WROOM-02

Commit message: up
Parts:
- added R5: 10k, esp32-dev-board:Register_0805_2012, symbol Device:R
Connections:
- net +3V3: now also R5.1
- net GPIO8: now also R5.2
Other:
- title: (none) -> ESP32C3DevBoard
Changed lines of the file:
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@@
 (kicad_sch (version 20211123) (generator eeschema)
   (paper "A4")
+  (title_block
+    (title "ESP32C3DevBoard")
+    (rev "v1.1.0")
+  )
   (junction (at 115.57 58.42) (diameter 0) (color 0 0 0 0)
   )
@@
   (junction (at 125.73 81.28) (diameter 0) (color 0 0 0 0)
   )
+  (junction (at 29.21 153.67) (diameter 0) (color 0 0 0 0)
+  )
   (junction (at 147.32 81.28) (diameter 0) (color 0 0 0 0)
   )
@@
     (stroke (width 0) (type default) (color 0 0 0 0))
   )
+  (wire (pts (xy 29.21 153.67) (xy 60.96 153.67))
+    (stroke (width 0) (type default) (color 0 0 0 0))
+  )
   (wire (pts (xy 81.28 81.28) (xy 81.28 85.09))
     (stroke (width 0) (type default) (color 0 0 0 0))
@@
   )
   (wire (pts (xy 115.57 71.12) (xy 115.57 78.74))
+    (stroke (width 0) (type default) (color 0 0 0 0))
+  )
+  (wire (pts (xy 25.4 153.67) (xy 29.21 153.67))
     (stroke (width 0) (type default) (color 0 0 0 0))
   )
@@
     )
   )
-  (global_label "GPIO8" (shape input) (at 60.96 153.67 180) (fields_autoplaced)
+  (global_label "GPIO8" (shape input) (at 25.4 153.67 180) (fields_autoplaced)
     (effects (font (size 1.27 1.27)) (justify right))
-    (property "シート間のリファレンス" "${INTERSHEET_REFS}" (id 0) (at 52.8621 153.7494 0)
+    (property "シート間のリファレンス" "${INTERSHEET_REFS}" (id 0) (at 17.3021 153.7494 0)
       (effects (font (size 1.27 1.27)) (justify right) hide)
     )
@@
     (pin "5")
     (pin "6")
+  )
+  (symbol (lib_id "Device:R") (at 29.21 149.86 0) (unit 1)
+    (in_bom yes) (on_board yes) (fields_autoplaced)
+    (property "Reference" "R5" (id 0) (at 31.75 148.5899 0)
+      (effects (font (size 1.27 1.27)) (justify left))
+    )
+    (property "Value" "10k" (id 1) (at 31.75 151.1299 0)
+      (effects (font (size 1.27 1.27)) (justify left))
+    )
+    (property "Footprint" "esp32-dev-board:Register_0805_2012" (id 2) (at 27.432 149.86 90)
+      (effects (font (size 1.27 1.27)) hide)
+    )
+    (property "Datasheet" "~" (id 3) (at 29.21 149.86 0)
+      (effects (font (size 1.27 1.27)) hide)
+    )
+    (pin "1")
+    (pin "2")
   )
   (symbol (lib_id "Device:C") (at 135.89 85.09 0) (unit 1)
@@
     (pin "1")
   )
+  (symbol (lib_id "power:+3V3") (at 29.21 146.05 0) (unit 1)
+    (in_bom yes) (on_board yes) (fields_autoplaced)
+    (property "Reference" "#PWR021" (id 0) (at 29.21 149.86 0)
+      (effects (font (size 1.27 1.27)) hide)
+    )
+    (property "Value" "+3V3" (id 1) (at 29.21 140.97 0))
+    (property "Footprint" "" (id 2) (at 29.21 146.05 0)
+      (effects (font (size 1.27 1.27)) hide)
+    )
+    (property "Datasheet" "" (id 3) (at 29.21 146.05 0)
+      (effects (font (size 1.27 1.27)) hide)
+    )
+    (pin "1")
+  )
   (sheet_instances
     (path "/" (page "1"))
@@
       (reference "#PWR020") (unit 1) (value "GND") (footprint "")
     )
+    (path "/fc65146f-31de-4f3b-a678-0e5eb0846754"
+      (reference "#PWR021") (unit 1) (value "+3V3") (footprint "")
+    )
     (path "/7f246871-c03d-457e-b71d-eba83974b239"
       (reference "C1") (unit 1) (value "10u") (footprint "esp32-dev-board:Capacitor_0805_2012")
@@
       (reference "R4") (unit 1) (value "5.1k") (footprint "esp32-dev-board:Register_0805_2012")
     )
+    (path "/7c15e983-d86d-4112-8b09-d22a0e2aa9db"
+      (reference "R5") (unit 1) (value "10k") (footprint "esp32-dev-board:Register_0805_2012")
+    )
     (path "/c41cfd04-4f71-4efe-908b-937fb32ea98e"

Commit message: update
Other:
- note added: "ESP32-C3 Module"
- note added: "Pinout"
- note added: "Power"
- note added: "Programing Port"
- note added: "USB"
- moved on the sheet: C1, C2, C3, C4, C5, C6, C7, D1, J1, J2, J3, J4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

Commit message: esp3s-c3-devboard/v1.2.0
Parts:
- removed J1: ESP32-C3-DEVKITC-02-J1, esp32-dev-board:ESP32-C3-DEVKITC-J1, symbol esp32-dev-board:ESP32-C3-DEVKITC-02-J1
- removed J2: ESP32-C3-DEVKITC-02-J2, esp32-dev-board:ESP32-C3-DEVKITC-J2, symbol esp32-dev-board:ESP32-C3-DEVKITC-02-J2
- removed J3: ESPProg-UART, esp32-dev-board:BoxPinHeader_2x03_P1.27mm_Vertical, symbol esp32-dev-board:ESPProg-UART
- added CH1, CH2: Pin_10, 74th:PinOut_Pin_10, symbol 74th_Interface:Pin_10
- added D2: PMEG2010ER,115, 74th:Package_SOD123W, symbol Device:D
- added J1: ESP-Prog-ProgramCOM_RECV, 74th:Connector_BoxPinHeader_2x03_P1.27mm, symbol 74th_Interface:ESP-Prog-ProgramCOM_RECV
- added R2, R4: 10, 74th:Register_0603_1608, symbol Device:R
- C1: renamed from C7; footprint esp32-dev-board:Capacitor_0805_2012 -> 74th:Capacitor_0603_1608
- C2: renamed from C6; footprint esp32-dev-board:Capacitor_0805_2012 -> 74th:Capacitor_0603_1608
- C3: renamed from C5; footprint esp32-dev-board:Capacitor_0805_2012 -> 74th:Capacitor_0603_1608
- C4: renamed from C3; footprint esp32-dev-board:Capacitor_0805_2012 -> 74th:Capacitor_0603_1608
- C5: renamed from C4; footprint esp32-dev-board:Capacitor_0805_2012 -> 74th:Capacitor_0603_1608
- C6: renamed from C1; footprint esp32-dev-board:Capacitor_0805_2012 -> 74th:Capacitor_0603_1608
- C7: renamed from C2; footprint esp32-dev-board:Capacitor_0805_2012 -> 74th:Capacitor_0603_1608
- D1: footprint LED_SMD:LED_0805_2012Metric_Pad1.15x1.40mm_HandSolder -> 74th:LED_0805_2012
- J2: renamed from J4; footprint esp32-dev-board:USB-C-12-Pin-MidMount-ali-v4 -> 74th:Connector_USB-C-Receptacle_SMT_12-Pin_Simple; symbol esp32-dev-board:USB2.0_C -> 74th_Interface:USB_TypeC-2.0_Receptacle
- R1: renamed from R2; footprint esp32-dev-board:Register_0805_2012 -> 74th:Register_0603_1608
- R3: renamed from R5; footprint esp32-dev-board:Register_0805_2012 -> 74th:Register_0603_1608
- R5: renamed from R1; footprint esp32-dev-board:Register_0805_2012 -> 74th:Register_0603_1608
- R6: renamed from R4; footprint esp32-dev-board:Register_0805_2012 -> 74th:Register_0603_1608
- R7: renamed from R3; footprint esp32-dev-board:Register_0805_2012 -> 74th:Register_0603_1608
- SW1: renamed from SW2; footprint esp32-dev-board:SKRPABE010 -> 74th:Switch_SKRPABE010
- SW2: renamed from SW1; footprint esp32-dev-board:SKRPABE010 -> 74th:Switch_SKRPABE010
- U1: renamed from U2; footprint esp32-dev-board:ESP32-C3-WROOM-02-handsolder -> PCM_Espressif:ESP32-C3-WROOM-02
- U2: renamed from U1; footprint Package_TO_SOT_SMD:SOT-223-3_TabPin2 -> 74th:Package_SOT-223-3; symbol Regulator_Linear:AMS1117-3.3 -> 74th_Passive:AMS1117-3.3_Regulator_SOT223
Connections:
- net +3V3: now also R5.1, CH1.1
- net +5V: now also CH1.9, D2.1 (K), J1.2 (VCC); no longer J2.1 (VBUS), R5.1
- net EN: now also CH1.2, J1.1 (EN)
- net GND: now also CH1.10, CH2.1, J1.4 (GND)
- net GPIO0 renamed IO0
- net IO0: now also CH2.2
- net GPIO1 renamed IO1
- net IO1: now also CH2.3
- net GPIO10 renamed IO10
- net IO10: now also CH2.10
- net GPIO18: no longer names the net of J2.2 (D-)
- net GPIO18: now also R4.1; no longer U1.13 (GPIO18/USB_D-)
- net GPIO19: no longer names the net of J2.3 (D+)
- net GPIO19: now also R2.1; no longer U1.14 (GPIO19/USB_D+)
- net GPIO2 renamed IO2
- net IO2: now also CH2.4
- net GPIO20 renamed IO20
- net IO20: now also CH2.9, J1.5 (RXD0)
- net GPIO21 renamed IO21
- net IO21: now also CH2.8, J1.3 (TXD0)
- net GPIO3 renamed IO3
- net IO3: now also CH2.5
- net GPIO4 renamed IO4
- net IO4: now also CH1.3
- net GPIO5 renamed IO5
- net IO5: now also CH1.4
- net GPIO6 renamed IO6
- net IO6: now also CH1.5
- net GPIO7 renamed IO7
- net IO7: now also CH1.6
- net GPIO8 renamed IO8
- net IO8: now also CH1.7
- net GPIO9 renamed IO9
- net IO9: now also CH1.8, J1.6 (IO0)
- new net: D2.2 (A), J2.1 (VBUS)
- new net IO18: CH2.7, R4.2, U1.13 (GPIO18/USB_D-)
- new net IO19: CH2.6, R2.2, U1.14 (GPIO19/USB_D+)
Other:
- moved on the sheet: C1, C2, C3, C4, C5, C6, C7, D1, R1, R3, R5, SW1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

Commit message: esp3s-c3-devboard/v1.2.1
Changed lines of the file:
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@@
 (kicad_sch
-	(version 20231120)
+	(version 20250114)
 	(generator "eeschema")
-	(generator_version "8.0")
+	(generator_version "9.0")
 	(paper "A4")
 	(title_block
 		(title "ESP32C3DevBoard")
-		(rev "v1.2.0")
+		(rev "v1.2.1")
+	)
+	(rectangle
+		(start 223.52 93.98)
+		(end 284.48 162.56)
+		(stroke
+			(width 0)
+			(type default)
+		)
+		(fill
+			(type none)
+		)
+	)
+	(rectangle
+		(start 137.16 93.98)
+		(end 223.52 162.56)
+		(stroke
+			(width 0)
+			(type default)
+		)
+		(fill
+			(type none)
+		)
+	)
+	(rectangle
+		(start 201.93 12.7)
+		(end 284.48 93.98)
+		(stroke
+			(width 0)
+			(type default)
+		)
+		(fill
+			(type none)
+		)
+	)
+	(rectangle
+		(start 12.7 12.7)
+		(end 137.16 162.56)
+		(stroke
+			(width 0)
+			(type default)
+		)
+		(fill
+			(type none)
+		)
+	)
+	(rectangle
+		(start 137.16 12.7)
+		(end 201.93 93.98)
+		(stroke
+			(width 0)
+			(type default)
+		)
+		(fill
+			(type none)
+		)
+	)
+	(text "ESP32-C3 Module"
+		(exclude_from_sim no)
+		(at 13.97 17.78 0)
+		(effects
+			(font
+				(size 2.54 2.54)
+			)
+			(justify left bottom)
+		)
+	)
+	(text "Pinout"
+		(exclude_from_sim no)
+		(at 138.43 99.06 0)
+		(effects
+			(font
+				(size 2.54 2.54)
+			)
+			(justify left bottom)
+		)
+	)
+	(text "Programing Port"
+		(exclude_from_sim no)
+		(at 224.79 99.06 0)
+		(effects
+			(font
+				(size 2.54 2.54)
+			)
+			(justify left bottom)
+		)
+	)
+	(text "Power"
+		(exclude_from_sim no)
+		(at 203.2 17.78 0)
+		(effects
+			(font
+				(size 2.54 2.54)
+			)
+			(justify left bottom)
+		)
+	)
+	(text "USB"
+		(exclude_from_sim no)
+		(at 138.43 17.78 0)
+		(effects
+			(font
+				(size 2.54 2.54)
+			)
+			(justify left bottom)
+		)
 	)
 	(junction
@@
 		)
 	)
-	(rectangle
-		(start 223.52 93.98)
-		(end 284.48 162.56)
-		(stroke
-			(width 0)
-			(type default)
-		)
-		(fill
-			(type none)
-		)
-	)
-	(rectangle
-		(start 137.16 93.98)
-		(end 223.52 162.56)
-		(stroke
-			(width 0)
-			(type default)
-		)
-		(fill
-			(type none)
-		)
-	)
-	(rectangle
-		(start 201.93 12.7)
-		(end 284.48 93.98)
-		(stroke
-			(width 0)
-			(type default)
-		)
-		(fill
-			(type none)
-		)
-	)
-	(rectangle
-		(start 12.7 12.7)
-		(end 137.16 162.56)
-		(stroke
-			(width 0)
-			(type default)
-		)
-		(fill
-			(type none)
-		)
-	)
-	(rectangle
-		(start 137.16 12.7)
-		(end 201.93 93.98)
-		(stroke
-			(width 0)
-			(type default)
-		)
-		(fill
-			(type none)
-		)
-	)
-	(text "ESP32-C3 Module"
-		(exclude_from_sim no)
-		(at 13.97 17.78 0)
-		(effects
-			(font
-				(size 2.54 2.54)
-			)
-			(justify left bottom)
-		)
-	)
-	(text "Pinout"
-		(exclude_from_sim no)
-		(at 138.43 99.06 0)
-		(effects
-			(font
-				(size 2.54 2.54)
-			)
-			(justify left bottom)
-		)
-	)
-	(text "Programing Port"
-		(exclude_from_sim no)
-		(at 224.79 99.06 0)
-		(effects
-			(font
-				(size 2.54 2.54)
-			)
-			(justify left bottom)
-		)
-	)
-	(text "Power"
-		(exclude_from_sim no)
-		(at 203.2 17.78 0)
-		(effects
-			(font
-				(size 2.54 2.54)
-			)
-			(justify left bottom)
-		)
-	)
-	(text "USB"
-		(exclude_from_sim no)
-		(at 138.43 17.78 0)
-		(effects
-			(font
-				(size 2.54 2.54)
-			)
-			(justify left bottom)
-		)
-	)
 	(label "IO19"
 		(at 204.47 132.08 180)
-		(fields_autoplaced yes)
 		(effects
 			(font
@@
 	(label "EN"
 		(at 260.35 140.97 180)
-		(fields_autoplaced yes)
 		(effects
 			(font
@@
 	(label "IO20"
 		(at 260.35 135.89 180)
-		(fields_autoplaced yes)
 		(effects
 			(font
@@
 	(label "IO18"
 		(at 204.47 134.62 180)
-		(fields_autoplaced yes)
 		(effects
 			(font
@@
 	(label "IO7"
 		(at 161.29 132.08 0)
-		(fields_autoplaced yes)
 		(effects
 			(font
@@
 	(label "IO4"
 		(at 57.15 80.01 0)
-		(fields_autoplaced yes)
 		(effects
 			(font
@@
 	(label "IO9"
 		(at 161.29 137.16 0)
-		(fields_autoplaced yes)
 		(effects
 			(font
@@
 	(label "IO8"
 		(at 161.29 134.62 0)
-		(fields_autoplaced yes)
 		(effects
 			(font
@@
 	(label "IO6"
 		(at 57.15 90.17 0)
-		(fields_autoplaced yes)
 		(effects
 			(font
@@
 	(label "IO3"
 		(at 204.47 129.54 180)
-		(fields_autoplaced yes)
 		(effects
 			(font
@@
 	(label "IO21"
 		(at 132.08 72.39 180)
-		(fields_autoplaced yes)
 		(effects
 			(font
@@
 	(label "IO2"
 		(at 204.47 127 180)
-		(fields_autoplaced yes)
 		(effects
 			(font
@@
 	(label "IO0"
 		(at 57.15 69.85 0)
-		(fields_autoplaced yes)
 		(effects
 			(font
@@
 	(label "IO9"
 		(at 260.35 138.43 180)
-		(fields_autoplaced yes)
 		(effects
 			(font
@@
 	(label "EN"
 		(at 57.15 64.77 0)
-		(fields_autoplaced yes)
 		(effects
 			(font
@@
 	(label "IO21"
 		(at 204.47 137.16 180)
-		(fields_autoplaced yes)
 		(effects
 			(font
@@
 	(label "IO4"
 		(at 161.29 124.46 0)
-		(fields_autoplaced yes)
 		(effects
 			(font
@@
 	(label "IO19"
 		(at 132.08 80.01 180)
-		(fields_autoplaced yes)
 		(effects
 			(font
@@
 	(label "IO7"
 		(at 57.15 92.71 0)
-		(fields_autoplaced yes)
 		(effects
 			(font
@@
 	(label "IO8"
 		(at 57.15 95.25 0)
-		(fields_autoplaced yes)
 		(effects
 			(font
@@
 	(label "IO6"
 		(at 161.29 129.54 0)
-		(fields_autoplaced yes)
 		(effects
 			(font
@@
 	(label "IO3"
 		(at 57.15 77.47 0)
-		(fields_autoplaced yes)
 		(effects
 			(font
@@
 	(label "IO10"
 		(at 204.47 142.24 180)
-		(fields_autoplaced yes)
 		(effects
 			(font
@@
 	(label "IO2"
 		(at 57.15 74.93 0)
-		(fields_autoplaced yes)
 		(effects
 			(font
@@
 	(label "IO18"
 		(at 132.08 77.47 180)
-		(fields_autoplaced yes)
 		(effects
 			(font
@@
 	(label "IO10"
 		(at 57.15 100.33 0)
-		(fields_autoplaced yes)
 		(effects
 			(font
@@
 	(label "IO1"
 		(at 57.15 72.39 0)
-		(fields_autoplaced yes)
 		(effects
 			(font
@@
 	(label "EN"
 		(at 161.29 121.92 0)
-		(fields_autoplaced yes)
 		(effects
 			(font
@@
 	(label "IO9"
 		(at 57.15 97.79 0)
-		(fields_autoplaced yes)
 		(effects
 			(font
@@
 	(label "IO20"
 		(at 204.47 139.7 180)
-		(fields_autoplaced yes)
 		(effects
 			(font
@@
 	(label "IO5"
 		(at 57.15 82.55 0)
-		(fields_autoplaced yes)
 		(effects
 			(font
@@
 	(label "IO19"
 		(at 195.58 50.8 180)
-		(fields_autoplaced yes)
 		(effects
 			(font
@@
 	(label "IO1"
 		(at 204.47 124.46 180)
-		(fields_autoplaced yes)
 		(effects
 			(font
@@
 	(label "IO20"
 		(at 132.08 69.85 180)
-		(fields_autoplaced yes)
 		(effects
 			(font
@@
 	(label "IO5"
 		(at 161.29 127 0)
-		(fields_autoplaced yes)
 		(effects
 			(font
@@
 	(label "IO0"
 		(at 204.47 121.92 180)
-		(fields_autoplaced yes)
 		(effects
 			(font
@@
 	(label "IO18"
 		(at 195.58 39.37 180)
-		(fields_autoplaced yes)
 		(effects
 			(font
@@
 	(label "IO21"
 		(at 260.35 133.35 180)
-		(fields_autoplaced yes)
 		(effects
 			(font
@@
 		)
 	)
+	(embedded_fonts no)
 )
