File: ESP32-Writer-CH340X/ESP32-Writer-CH340X.kicad_sch (KiCad schematic)
At the start: 7 parts, among them J1 ESP-Prog-ProgramCOM-SEND, J2 USB2.0_C_v3, U1 CH340X

Commit message: update Document
Parts:
- R3: value 4.3k -> 4.7k
Changed lines of the file:
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@@
       (effects (font (size 1.27 1.27)) (justify left))
     )
-    (property "Value" "4.3k" (at 149.86 70.485 0)
+    (property "Value" "4.7k" (at 149.86 70.485 0)
       (effects (font (size 1.27 1.27)) (justify left))
     )
