File: ESP32-WROOM-32/ESP32-WROOM-32.kicad_pcb (KiCad board)
At the start: 2 copper layers, 25.4 x 34.3 mm, 21 parts, among them J1 USB2.0_C_v3, J4 ESP-Prog-ProgramCOM-RECV, SW1 BT, SW2 RST, U2 AMS1117-3.3, U3 ESP32-WROOM-32D

Commit message: esp32-wroom-32/v1.0.0
Parts:
- added G***: LOGO, $74th:74th-5mm, B.Cu at (73.3, 61.0)
- added REF**: twitter, $74th:twitter, B.Cu at (73.3, 57.5)
- moved C6 0.25 mm to (74.9, 45.3)
- moved D1 0.11 mm to (72.3, 66.7)
Routing:
- net EN: track 0.00 -> 84.5 mm, vias 0 -> 1
- net GPIO0: track 0.00 -> 56.7 mm
- net GND: track 0.00 -> 54.3 mm, vias 0 -> 31
- net U0TXD: track 0.00 -> 46.9 mm, vias 0 -> 5
- net U0RXD: track 0.00 -> 46.3 mm, vias 0 -> 2
- net GPIO12: track 0.00 -> 37.8 mm, vias 0 -> 1
- net GPIO2: track 0.00 -> 33.3 mm, vias 0 -> 1
- net +5V: track 13.2 -> 43.9 mm, vias 0 -> 2
- net GPIO14: track 0.00 -> 26.9 mm, vias 0 -> 3
- net GPIO22: track 0.00 -> 25.9 mm, vias 0 -> 1
- net GPIO21: track 0.00 -> 25.7 mm, vias 0 -> 1
- net GPIO4: track 0.00 -> 25.7 mm, vias 0 -> 1
- net GPIO23: track 0.00 -> 25.6 mm
- net GPIO19: track 0.00 -> 20.3 mm, vias 0 -> 1
- net GPIO33: track 0.00 -> 19.0 mm, vias 0 -> 1
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Other:
- board text added: "0"
- board text added: "12"
- board text added: "13"
- board text added: "14"
- board text added: "15"
- board text added: "18"
- board text added: "19"
- board text added: "2"
- board text added: "21"
- board text added: "22"
- board text added: "23"
- board text added: "25"
- board text added: "26"
- board text added: "27"
- board text added: "32"
- board text added: "33"
- board text added: "3V"
- board text added: "4"
- board text added: "5"
- board text added: "5V"
- board text added: "BOOT"
- board text added: "EN"
- board text added: "ESP32"
- board text added: "G"
- board text added: "Micro"
- board text added: "PWR"
- board text added: "R"
- board text added: "T"
- board text added: "v1.0.0"

Commit message: esp32-wroom-32/v1.0.0
Parts:
- renumbered C6 to C1, C5 to C2, C2 to C3, C3 to C5, D5 to D2, J4 to J1, J1 to J2, R4 to R1, R5 to R2, R1 to R4, R2 to R5, U3 to U1
Changed lines of the file:
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@@
     (property "ki_keywords" "LED diode")
     (attr smd)
-    (fp_text reference "D5" (at -0.245 1.778) (layer "F.SilkS")
+    (fp_text reference "D2" (at -0.245 1.778) (layer "F.SilkS")
         (effects (font (size 0.8 0.8) (thickness 0.12)))
     )
@@
     (property "ki_keywords" "usb universal serial bus type-C USB2.0")
     (attr smd)
-    (fp_text reference "J1" (at -0.01 -6.205 180) (layer "F.Fab") hide
+    (fp_text reference "J2" (at -0.01 -6.205 180) (layer "F.Fab") hide
         (effects (font (size 0.7 0.7) (thickness 0.15)))
     )
@@
     (property "ki_keywords" "RF Radio BT ESP ESP32 Espressif onboard PCB antenna")
     (attr smd)
-    (fp_text reference "U3" (at -0.013 2.545) (layer "F.SilkS")
+    (fp_text reference "U1" (at -0.013 2.545) (layer "F.SilkS")
         (effects (font (size 1 1) (thickness 0.15)))
     )
@@
     (property "Sheetname" "")
     (attr through_hole)
-    (fp_text reference "J4" (at 1.651 -3.048) (layer "F.SilkS")
+    (fp_text reference "J1" (at 1.651 -3.048) (layer "F.SilkS")
         (effects (font (size 1 1) (thickness 0.15)))
     )
@@
     (property "ki_keywords" "R res resistor")
     (attr smd)
-    (fp_text reference "R5" (at 0 -1.651) (layer "B.SilkS")
+    (fp_text reference "R2" (at 0 -1.651) (layer "B.SilkS")
         (effects (font (size 0.8 0.8) (thickness 0.12)) (justify mirror))
     )
@@
     (property "ki_keywords" "cap capacitor")
     (attr smd)
-    (fp_text reference "C5" (at -2.667 0) (layer "B.SilkS")
+    (fp_text reference "C2" (at -2.667 0) (layer "B.SilkS")
         (effects (font (size 0.8 0.8) (thickness 0.12)) (justify mirror))
     )
@@
     (property "ki_keywords" "cap capacitor")
     (attr smd)
-    (fp_text reference "C6" (at -2.667 0) (layer "B.SilkS")
+    (fp_text reference "C1" (at -2.667 0) (layer "B.SilkS")
         (effects (font (size 0.8 0.8) (thickness 0.12)) (justify mirror))
     )
@@
     (property "ki_keywords" "R res resistor")
     (attr smd)
-    (fp_text reference "R1" (at -1.254 -1.778) (layer "B.SilkS")
+    (fp_text reference "R4" (at -1.254 -1.778) (layer "B.SilkS")
         (effects (font (size 0.8 0.8) (thickness 0.12)) (justify mirror))
     )
@@
     (property "ki_keywords" "R res resistor")
     (attr smd)
-    (fp_text reference "R4" (at -2.794 0) (layer "B.SilkS")
+    (fp_text reference "R1" (at -2.794 0) (layer "B.SilkS")
         (effects (font (size 0.8 0.8) (thickness 0.12)) (justify mirror))
     )
@@
     (property "ki_keywords" "cap capacitor")
     (attr smd)
-    (fp_text reference "C3" (at 2.54 -0.127) (layer "B.SilkS")
+    (fp_text reference "C5" (at 2.54 -0.127) (layer "B.SilkS")
         (effects (font (size 0.8 0.8) (thickness 0.12)) (justify mirror))
     )
@@
     (property "ki_keywords" "cap capacitor")
     (attr smd)
-    (fp_text reference "C2" (at -2.794 0) (layer "B.SilkS")
+    (fp_text reference "C3" (at -2.794 0) (layer "B.SilkS")
         (effects (font (size 0.8 0.8) (thickness 0.12)) (justify mirror))
     )
@@
     (property "ki_keywords" "R res resistor")
     (attr smd)
-    (fp_text reference "R2" (at -0.365 -1.778) (layer "B.SilkS")
-        (effects (font (size 0.8 0.8) (thickness 0.12)) (justify mirror))
-    )
+    (fp_text reference "R5" (at -0.365 -1.778) (layer "B.SilkS")
+        (effects (font (size 0.8 0.8) (thickness 0.12)) (justify mirror))
+    )

Commit message: ESP32-WROOM32
Parts:
- added REF**: JLCJLCJLCJLC, $74th:JLCJLCJLCJLC, F.Cu at (80.3, 46.5)
