File: ESP32-WROOM-32/ESP32-WROOM-32.kicad_sch (KiCad schematic)
At the start: 21 parts, among them J3 USB2.0_C_v3, J4 ESP-Prog-ProgramCOM-RECV, SW1 BT, SW2 RST, U1 AMS1117-3.3, U3 ESP32-WROOM-32D

Commit message: esp32-wroom-32/v1.0.0
Parts:
- renumbered U3 to U1
Changed lines of the file:
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@@
       (project "ESP32-WROOM-32"
         (path "/25f0b93d-04b7-4f4a-9ab9-040076a6e73f"
-          (reference "J4") (unit 1)
+          (reference "J1") (unit 1)
         )
       )
@@
       (project "ESP32-WROOM-32"
         (path "/25f0b93d-04b7-4f4a-9ab9-040076a6e73f"
-          (reference "C3") (unit 1)
+          (reference "C5") (unit 1)
         )
       )
@@
       (project "ESP32-WROOM-32"
         (path "/25f0b93d-04b7-4f4a-9ab9-040076a6e73f"
-          (reference "R5") (unit 1)
+          (reference "R2") (unit 1)
         )
       )
@@
       (project "ESP32-WROOM-32"
         (path "/25f0b93d-04b7-4f4a-9ab9-040076a6e73f"
+          (reference "R5") (unit 1)
+        )
+      )
+    )
+  )
+  (symbol (lib_id "Device:C") (at 73.66 43.18 0) (unit 1)
+    (in_bom yes) (on_board yes) (dnp no) (fields_autoplaced)
+    (property "Reference" "C3" (at 77.47 41.9099 0)
+      (effects (font (size 1.27 1.27)) (justify left))
+    )
+    (property "Value" "100n" (at 77.47 44.4499 0)
+      (effects (font (size 1.27 1.27)) (justify left))
+    )
+    (property "Footprint" "$74th:Capacitor_0805_2012" (at 74.6252 46.99 0)
+      (effects (font (size 1.27 1.27)) hide)
+    )
+    (property "Datasheet" "~" (at 73.66 43.18 0)
+      (effects (font (size 1.27 1.27)) hide)
+    )
+    (pin "1")
+    (pin "2")
+    (instances
+      (project "ESP32-S3-WROOM-1"
+        (path "/1f0126c3-e865-4b7c-bf68-4d53d0d38c5a"
+          (reference "C3") (unit 1)
+        )
+      )
+      (project "ESP32-WROOM-32"
+        (path "/25f0b93d-04b7-4f4a-9ab9-040076a6e73f"
+          (reference "C4") (unit 1)
+        )
+      )
+    )
+  )
+  (symbol (lib_id "Switch:SW_Push") (at 185.42 91.44 0) (unit 1)
+    (in_bom yes) (on_board yes) (dnp no) (fields_autoplaced)
+    (property "Reference" "SW1" (at 185.42 83.82 0)
+      (effects (font (size 1.27 1.27)))
+    )
+    (property "Value" "BT" (at 185.42 86.36 0)
+      (effects (font (size 1.27 1.27)))
+    )
+    (property "Footprint" "$74th:SKRPABE010" (at 185.42 86.36 0)
+      (effects (font (size 1.27 1.27)) hide)
+    )
+    (property "Datasheet" "~" (at 185.42 86.36 0)
+      (effects (font (size 1.27 1.27)) hide)
+    )
+    (pin "1")
+    (pin "2")
+    (instances
+      (project "ESP32-S3-WROOM-1"
+        (path "/1f0126c3-e865-4b7c-bf68-4d53d0d38c5a"
+          (reference "SW1") (unit 1)
+        )
+      )
+      (project "ESP32-WROOM-32"
+        (path "/25f0b93d-04b7-4f4a-9ab9-040076a6e73f"
+          (reference "SW1") (unit 1)
+        )
+      )
+    )
+  )
+  (symbol (lib_id "Device:R") (at 43.18 71.12 0) (unit 1)
+    (in_bom yes) (on_board yes) (dnp no) (fields_autoplaced)
+    (property "Reference" "R2" (at 45.72 69.8499 0)
+      (effects (font (size 1.27 1.27)) (justify left))
+    )
+    (property "Value" "5.1k" (at 45.72 72.3899 0)
+      (effects (font (size 1.27 1.27)) (justify left))
+    )
+    (property "Footprint" "$74th:Register_0805_2012" (at 41.402 71.12 90)
+      (effects (font (size 1.27 1.27)) hide)
+    )
+    (property "Datasheet" "~" (at 43.18 71.12 0)
+      (effects (font (size 1.27 1.27)) hide)
+    )
+    (pin "1")
+    (pin "2")
+    (instances
+      (project "ESP32-S3-WROOM-1"
+        (path "/1f0126c3-e865-4b7c-bf68-4d53d0d38c5a"
           (reference "R2") (unit 1)
         )
       )
-    )
-  )
-  (symbol (lib_id "Device:C") (at 73.66 43.18 0) (unit 1)
-    (in_bom yes) (on_board yes) (dnp no) (fields_autoplaced)
-    (property "Reference" "C3" (at 77.47 41.9099 0)
-      (effects (font (size 1.27 1.27)) (justify left))
-    )
-    (property "Value" "100n" (at 77.47 44.4499 0)
-      (effects (font (size 1.27 1.27)) (justify left))
-    )
-    (property "Footprint" "$74th:Capacitor_0805_2012" (at 74.6252 46.99 0)
-      (effects (font (size 1.27 1.27)) hide)
-    )
-    (property "Datasheet" "~" (at 73.66 43.18 0)
-      (effects (font (size 1.27 1.27)) hide)
-    )
-    (pin "1")
-    (pin "2")
-    (instances
-      (project "ESP32-S3-WROOM-1"
-        (path "/1f0126c3-e865-4b7c-bf68-4d53d0d38c5a"
-          (reference "C3") (unit 1)
-        )
-      )
-      (project "ESP32-WROOM-32"
-        (path "/25f0b93d-04b7-4f4a-9ab9-040076a6e73f"
-          (reference "C4") (unit 1)
-        )
-      )
-    )
-  )
-  (symbol (lib_id "Switch:SW_Push") (at 185.42 91.44 0) (unit 1)
-    (in_bom yes) (on_board yes) (dnp no) (fields_autoplaced)
-    (property "Reference" "SW1" (at 185.42 83.82 0)
-      (effects (font (size 1.27 1.27)))
-    )
-    (property "Value" "BT" (at 185.42 86.36 0)
-      (effects (font (size 1.27 1.27)))
-    )
-    (property "Footprint" "$74th:SKRPABE010" (at 185.42 86.36 0)
-      (effects (font (size 1.27 1.27)) hide)
-    )
-    (property "Datasheet" "~" (at 185.42 86.36 0)
-      (effects (font (size 1.27 1.27)) hide)
-    )
-    (pin "1")
-    (pin "2")
-    (instances
-      (project "ESP32-S3-WROOM-1"
-        (path "/1f0126c3-e865-4b7c-bf68-4d53d0d38c5a"
-          (reference "SW1") (unit 1)
-        )
-      )
-      (project "ESP32-WROOM-32"
-        (path "/25f0b93d-04b7-4f4a-9ab9-040076a6e73f"
-          (reference "SW1") (unit 1)
-        )
-      )
-    )
-  )
-  (symbol (lib_id "Device:R") (at 43.18 71.12 0) (unit 1)
-    (in_bom yes) (on_board yes) (dnp no) (fields_autoplaced)
-    (property "Reference" "R2" (at 45.72 69.8499 0)
-      (effects (font (size 1.27 1.27)) (justify left))
-    )
-    (property "Value" "5.1k" (at 45.72 72.3899 0)
-      (effects (font (size 1.27 1.27)) (justify left))
-    )
-    (property "Footprint" "$74th:Register_0805_2012" (at 41.402 71.12 90)
-      (effects (font (size 1.27 1.27)) hide)
-    )
-    (property "Datasheet" "~" (at 43.18 71.12 0)
-      (effects (font (size 1.27 1.27)) hide)
-    )
-    (pin "1")
-    (pin "2")
-    (instances
-      (project "ESP32-S3-WROOM-1"
-        (path "/1f0126c3-e865-4b7c-bf68-4d53d0d38c5a"
-          (reference "R2") (unit 1)
-        )
-      )
-      (project "ESP32-WROOM-32"
-        (path "/25f0b93d-04b7-4f4a-9ab9-040076a6e73f"
-          (reference "R1") (unit 1)
+      (project "ESP32-WROOM-32"
+        (path "/25f0b93d-04b7-4f4a-9ab9-040076a6e73f"
+          (reference "R4") (unit 1)
         )
       )
@@
       (project "ESP32-WROOM-32"
         (path "/25f0b93d-04b7-4f4a-9ab9-040076a6e73f"
-          (reference "R4") (unit 1)
+          (reference "R1") (unit 1)
         )
       )
@@
       (project "ESP32-WROOM-32"
         (path "/25f0b93d-04b7-4f4a-9ab9-040076a6e73f"
-          (reference "C2") (unit 1)
+          (reference "C3") (unit 1)
         )
       )
@@
       (project "ESP32-WROOM-32"
         (path "/25f0b93d-04b7-4f4a-9ab9-040076a6e73f"
-          (reference "J1") (unit 1)
+          (reference "J2") (unit 1)
         )
       )
@@
   (symbol (lib_id "RF_Module:ESP32-WROOM-32D") (at 59.69 143.51 0) (unit 1)
     (in_bom yes) (on_board yes) (dnp no) (fields_autoplaced)
-    (property "Reference" "U3" (at 61.6459 106.68 0)
+    (property "Reference" "U1" (at 61.6459 106.68 0)
       (effects (font (size 1.27 1.27)) (justify left))
     )
@@
       (project "ESP32-WROOM-32"
         (path "/25f0b93d-04b7-4f4a-9ab9-040076a6e73f"
-          (reference "U3") (unit 1)
+          (reference "U1") (unit 1)
         )
       )
@@
       (project "ESP32-WROOM-32"
         (path "/25f0b93d-04b7-4f4a-9ab9-040076a6e73f"
-          (reference "C5") (unit 1)
+          (reference "C2") (unit 1)
         )
       )
@@
       (project "ESP32-WROOM-32"
         (path "/25f0b93d-04b7-4f4a-9ab9-040076a6e73f"
-          (reference "D5") (unit 1)
+          (reference "D2") (unit 1)
         )
       )
@@
       (project "ESP32-WROOM-32"
         (path "/25f0b93d-04b7-4f4a-9ab9-040076a6e73f"
-          (reference "C6") (unit 1)
-        )
-      )
+          (reference "C1") (unit 1)
+        )
+      )

Commit message: ESP32-WROOM32
Parts:
- D5: value PWR -> Blue
- D5: value PWR -> Red
- R4: value 10k -> 5.1k
Changed lines of the file:
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@@
   (symbol (lib_id "Device:R") (at 127 43.18 180) (unit 1)
     (in_bom yes) (on_board yes) (dnp no) (fields_autoplaced)
-    (property "Reference" "R4" (at 129.54 41.9099 0)
+    (property "Reference" "R4" (at 129.54 42.545 0)
       (effects (font (size 1.27 1.27)) (justify right))
     )
-    (property "Value" "10k" (at 129.54 44.4499 0)
+    (property "Value" "5.1k" (at 129.54 45.085 0)
       (effects (font (size 1.27 1.27)) (justify right))
     )
@@
   (symbol (lib_id "Device:LED") (at 92.71 129.54 90) (unit 1)
     (in_bom yes) (on_board yes) (dnp no) (fields_autoplaced)
-    (property "Reference" "D5" (at 96.52 129.8574 90)
+    (property "Reference" "D5" (at 96.52 130.4925 90)
       (effects (font (size 1.27 1.27)) (justify right))
     )
-    (property "Value" "PWR" (at 96.52 132.3974 90)
+    (property "Value" "Blue" (at 96.52 133.0325 90)
       (effects (font (size 1.27 1.27)) (justify right))
     )
@@
   (symbol (lib_id "Device:LED") (at 127 50.8 90) (unit 1)
     (in_bom yes) (on_board yes) (dnp no) (fields_autoplaced)
-    (property "Reference" "D5" (at 130.81 51.1174 90)
+    (property "Reference" "D5" (at 130.81 51.7525 90)
       (effects (font (size 1.27 1.27)) (justify right))
     )
-    (property "Value" "PWR" (at 130.81 53.6574 90)
+    (property "Value" "Red" (at 130.81 54.2925 90)
       (effects (font (size 1.27 1.27)) (justify right))
     )

Commit message: update
Other:
- note added: "Buttons"
- note added: "ESP32 Module"
- note added: "Pinout"
- note added: "Programing Port"
- note added: "USB & Power"
- company: (none) -> 74th
- title: (none) -> Mini ESP32 Dev Board
- moved on the sheet: C2, C3, C4, C5, C6, CH1, CH2, D1, D5, J3, J4, R2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
