File: ESP32-Writer-CH340G/ESP32-Writer-CH340G.kicad_pcb (KiCad board)
At the start: 2 copper layers, 50.8 x 31.1 mm, 34 parts, among them J1 ESP-Prog-ProgramCOM-SEND, J2 USB2.0_C, J3 UART-OUTPUT, J4 USB2.0_C, Q1 2N7002, Q2 2N7002, SW1 SK-12D02-G020, U1 AMS1117-3.3, U2 CH340G, Y1 12M

Commit message: update
Parts:
- removed C6, C7: 22p, 74th:Capacitor_0805_2012
- removed Y1: 12M, 74th:Crystal_SMD_3225-4Pin_3.2x2.5mm_HandSoldering
- added D3: PMEG2010ER, 74th:Package_SOD123W, F.Cu at (62.9, 52.1)
- J1: footprint $74th:BoxPinHeader_2x03_P1.27mm_Vertical -> 74th:Connector_BoxPinHeader_2x03_P1.27mm
- Q1, Q2: footprint Package_TO_SOT_SMD:SOT-23 -> 74th:Package_SOT-23
- R6, R7: footprint 74th:Capacitor_0805_2012 -> 74th:Register_0805_2012
- U1: footprint Package_TO_SOT_SMD:SOT-223-3_TabPin2 -> 74th:Package_SOT-223-3
- U2: value CH340G -> CH340C
- moved U2 2.41 mm to (69.8, 55.1)
- moved C3 1.73 mm to (76.2, 55.9)
Connections:
- F2 pad 2: +5V -> Net-(D3-A)
- U2 pad 7: Net-(U2-XI) -> unconnected-(U2-NC-Pad7)
- U2 pad 8: Net-(U2-XO) -> unconnected-(U2-OUT-Pad8)
- U2 pad 9: unconnected-(U2-CTS-Pad9) -> (no net)
Routing:
- net Net-(U2-XO): track 9.17 -> 0.00 mm
- net Net-(U2-XI): track 5.88 -> 0.00 mm
- net GND: track 16.7 -> 10.8 mm, vias 99 -> 95
- net unconnected-(J2-D+-Pad3)_0: track 5.21 -> 0.00 mm
- net unconnected-(J2-D+-Pad3): track 0.00 -> 5.21 mm
- net Net-(U2-V3): track 4.88 -> 0.00 mm
- net /DM: track 12.4 -> 15.2 mm
- net Net-(D3-A): track 0.00 -> 2.80 mm
- net /DP: track 13.3 -> 15.7 mm
- net /DTR: track 23.9 -> 21.6 mm
- net Net-(D2-K): track 30.1 -> 28.0 mm
- net VCC: track 16.9 -> 18.6 mm
- net Net-(D2-A): track 19.2 -> 17.8 mm
- net +5V: track 90.4 -> 89.8 mm
Other:
- board size 50.8 x 31.1 mm -> 54.6 x 31.1 mm
