File: ESP32-H2-MINI-1/basic/ESP32-H2-MINI-1-basic.kicad_pcb (KiCad board)
At the start: 2 copper layers, 30.5 x 35.6 mm, 44 parts, among them J1 ESP-Prog-ProgramCOM_RECV, J2 USB2.0-C_SMT, M1 Hole_M2_2.0, M2 Hole_M2_2.0, M3 Hole_M2_2.0, M4 Hole_M2_2.0, M5 Hole_M2_2.0, SW1 SW_Push, SW2 SW_Push, U1 ESP32-H2-MINI-1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

Commit message: small fix
Parts:
- removed M4 (x2): Hole_M2_2.0, 74th:Hole_M2_2.0
- C4, C5: value 10p -> 12p
- R1, R2: value 27 -> 10
- Y1: footprint 74th:Crystal_SMD_2012-2Pin_2.0x1.2mm_HandSoldering -> 74th:Crystal_SMD_3215-2Pin_3.2x1.5mm
- mouse-bite-1 (x2), mouse-bite-2 (x2): footprint $74th:mouse-bite-1.27mm-slot -> 74th:MouseBite_1.27mm_slot_half
- moved C5 0.33 mm to (143.3, 42.1)
- moved C7 0.32 mm to (140.8, 48.8)
- moved C6 0.29 mm to (140.8, 47.3)
- moved Y1 0.24 mm to (142.7, 45.1), turned to 0 degrees
- moved C4 0.20 mm to (141.7, 42.2)
- moved C3 0.13 mm to (141.7, 39.8)
- turned mouse-bite-1 to -90 degrees
- turned mouse-bite-2 to -90 degrees
Routing:
- net /GPIO13-XTAL: track 4.21 -> 7.90 mm
- net /GPIO14-XTAL: track 5.83 -> 7.81 mm
- net /GPIO12: track 12.5 -> 13.6 mm
- net VBAT: track 31.2 -> 31.7 mm
- net +3V3: track 41.8 -> 42.3 mm
- net GND: track 112.7 -> 113.2 mm, vias 64 -> 63
Other:
- outline, holes or cut-outs redrawn
- board text added: "3V"
- board text added: "74th-G047-v1.0.1"
- board text removed: "3v"
- board text removed: "74th-G047-v1.0.0"
