File: ESP32-H2-MINI-1/basic/ESP32-H2-MINI-1-basic.kicad_sch (KiCad schematic)
At the start: 28 parts, among them J1 ESP-Prog-ProgramCOM_RECV, J2 USB2.0-C_SMT, SW1 SW_Push, SW2 SW_Push, U1 ESP32-H2-MINI-1, U2 AMS1117, Y1 32k

Commit message: small fix
Parts:
- C4, C5: value 10p -> 12p
- R1, R2: value 27 -> 10
- Y1: footprint 74th:Crystal_SMD_2012-2Pin_2.0x1.2mm_HandSoldering -> 74th:Crystal_SMD_3215-2Pin_3.2x1.5mm
Changed lines of the file:
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@@
 			)
 		)
-		(property "Value" "27"
+		(property "Value" "10"
 			(at 147.828 58.42 90)
 			(effects
@@
 			)
 		)
-		(property "Footprint" "74th:Crystal_SMD_2012-2Pin_2.0x1.2mm_HandSoldering"
+		(property "Footprint" "74th:Crystal_SMD_3215-2Pin_3.2x1.5mm"
 			(at 45.72 130.81 0)
 			(effects
@@
 			)
 		)
-		(property "Value" "10p"
+		(property "Value" "12p"
 			(at 35.56 119.38 90)
 			(effects
@@
 			)
 		)
-		(property "Value" "10p"
+		(property "Value" "12p"
 			(at 35.56 132.08 90)
 			(effects
@@
 			)
 		)
-		(property "Value" "27"
+		(property "Value" "10"
 			(at 148.082 64.77 90)
 			(effects
