File: ESP32-C6-WROOM-1/ESP32-C6-WROOM-1.kicad_sch (KiCad schematic)
At the start: 22 parts, among them J1 ESP-Prog-ProgramCOM_RECV, J2 USB2.0-C_SMT, SW1 SW_Push, SW2 SW_Push, U1 ESP32-C6-WROOM-1, U2 AMS1117

Commit message: small fix
Parts:
- R2, R3: value 27 -> 10
Changed lines of the file:
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@@
 			)
 		)
-		(property "Value" "27"
+		(property "Value" "10"
 			(at 111.76 53.34 90)
 			(effects
@@
 			)
 		)
-		(property "Value" "27"
+		(property "Value" "10"
 			(at 111.76 63.5 90)
 			(effects
