File: ESP-Writer-CH9102F/ESP-Writer-CH9102F.kicad_pcb (KiCad board)
At the start: 2 copper layers, 34.2 x 19.5 mm, 31 parts, among them J1 USB2.0-C_SMT, J2 ESP-Prog-ProgramCOM_SEND, SW1 SW_Push, U1 CH9102F, U2 CH32V003J4M6, U3 CH213K, U4 AMS1117

Commit message: esp32-writer-ch9102f
Parts:
- added MISC-ICON: LOGO, 74th:Logo_74th_4mm, B.Cu at (77.5, 36.2)
Other:
- board text added: "/3V3"
- board text added: "BT"
- board text added: "EN"
- board text added: "ESP32Writer"
- board text added: "GND"
- board text added: "RXD"
- board text added: "TXD"
- board text removed: "/3.3V"
- board text removed: "ESP-Writer"
