File: ESP32-Writer-CH9102F/ESP-Writer-CH9102F.kicad_pcb (KiCad board)
At the start: 2 copper layers, 34.2 x 19.5 mm, 32 parts, among them J1 USB2.0-C_SMT, J2 ESP-Prog-ProgramCOM_SEND, SW1 SW_Push, U1 CH9102F, U2 CH32V003J4M6, U3 CH213K, U4 AMS1117

Commit message: esp32-writer-ch9102f/v1.1.0
Parts:
- removed CH2: SWD, 74th:PinOut_Pin_2
- removed D4: YELLOW, 74th:LED_0805_2012
- removed R6: 1k, 74th:Register_0603_1608
- removed R7: 10k, 74th:Register_0603_1608
- removed R8, R9: 10, 74th:Register_0603_1608
- removed SW1: SW_Push, 74th:Switch_SKRPABE010_Pin-4
- removed U2: CH32V003J4M6, 74th:Package_SOIC-8_3.9x4.9mm_P1.27mm
- added Q1: 2N7002, 74th:Package_SOT-23, B.Cu at (65.2, 43.0)
- added Q2: 2N7002, 74th:Package_SOT-23, B.Cu at (60.8, 43.0)
- C5: value 100n -> 22u; moved to B.Cu
- F1: value Polyfuse -> KT6-1100SMDI
- moved C5 9.40 mm to (69.9, 42.1), turned to 180 degrees
Connections:
- C5 pad 1: VDD -> Net-(J2-VCC)
Routing:
- net GND: track 38.7 -> 25.4 mm, vias 65 -> 62
- net Net-(U2-PC1): track 10.8 -> 0.00 mm, vias 2 -> 0
- net /SWDIO: track 10.5 -> 0.00 mm, vias 1 -> 0
- net Net-(R7-Pad1): track 9.69 -> 0.00 mm, vias 2 -> 0
- net /DTR: track 18.7 -> 27.5 mm
- net /ESP_BOOT: track 15.1 -> 23.7 mm
- net Net-(U2-PC4): track 7.35 -> 0.00 mm, vias 1 -> 0
- net Net-(U2-PC2): track 6.29 -> 0.00 mm, vias 2 -> 0
- net /ESP_EN: track 10.8 -> 15.7 mm
- net VDD: track 88.7 -> 84.9 mm, vias 11 -> 9
- net Net-(D4-K): track 2.50 -> 0.00 mm, vias 1 -> 0
- net +5V: track 73.4 -> 74.0 mm
- net Net-(J2-VCC): track 13.6 -> 13.4 mm, vias 1 -> 2
Other:
- board text removed: "CH32VSWD"
- board text removed: "D"
- board text removed: "G"
